File: kicad/FPGA.sch (KiCad schematic (older format))
At the start: 51 parts, among them U3 MCP4725

Commit message: Layout [in progress]
Parts:
- added R8, R9: 4.7k, Resistors_SMD:R_0603_HandSoldering, symbol R
Connections:
- net +3V3: now also R8.1, R9.1
- net SCL_DAC: now also R8.2
- net SDA_DAC: now also R9.2

Commit message: Layout [in progress]
Connections:
- no-connect marks 75 -> 77
Changed lines of the file:
@@
 L +1.2V #PWR030
 U 1 1 595F9456
-P 9500 1600
-F 0 "#PWR030" H 9500 1740 20  0001 C CNN
-F 1 "+1.2V" H 9500 1710 30  0000 C CNN
-F 2 "" H 9500 1600 60  0000 C CNN
-F 3 "" H 9500 1600 60  0000 C CNN
-	1    9500 1600
+P 9500 1575
+F 0 "#PWR030" H 9500 1715 20  0001 C CNN
+F 1 "+1.2V" H 9500 1685 30  0000 C CNN
+F 2 "" H 9500 1575 60  0000 C CNN
+F 3 "" H 9500 1575 60  0000 C CNN
+	1    9500 1575
 	1    0    0    -1
 $EndComp
@@
 	9300 1625 9300 1675
 Wire Wire Line
-	9500 1600 9500 1675
+	9500 1575 9500 1675
 Wire Wire Line
 	9100 975  9100 925
@@
 Wire Wire Line
 	8900 1625 9500 1625
-$Comp
-L xc6slx9_144 xc6slx9_1
-U 7 1 595EA267
-P 8750 1400
-F 0 "xc6slx9_1" H 8625 1750 50  0000 C CNN
-F 1 "xc6slx9_144" H 8600 1825 50  0000 C CNN
-F 2 "Housings_QFP:TQFP-144_20x20mm_Pitch0.5mm" H 8975 2125 60  0001 C CNN
-F 3 "" H 8975 2125 60  0001 C CNN
-	7    8750 1400
-	1    0    0    -1
-$EndComp
 Wire Wire Line
 	8900 1425 8950 1425
@@
 	4400 1675 4400 1850
 Connection ~ 4400 1850
+NoConn ~ 8900 3850
+NoConn ~ 8900 3950
+$Comp
+L xc6slx9_144 xc6slx9_1
+U 7 1 595EA267
+P 8750 1400
+F 0 "xc6slx9_1" H 8625 1750 50  0000 C CNN
+F 1 "xc6slx9_144" H 8600 1825 50  0000 C CNN
+F 2 "Housings_QFP:TQFP-144_20x20mm_Pitch0.5mm" H 8975 2125 60  0001 C CNN
+F 3 "" H 8975 2125 60  0001 C CNN
+	7    8750 1400
+	1    0    0    -1
+$EndComp
+Connection ~ 8950 1425
 $EndSCHEMATC

Commit message: layout [in progress]
Parts:
- added D11: LED, Footprints_LJ:Mini_TopLed_SMD, symbol LED
- added R39: 680R, Resistors_SMD:R_0603_HandSoldering, symbol R
- added X1: Stiftleiste_2x10Pm_R2.54, Footprints_LJ:Stiftleiste_2x10Pm_R2.54, symbol Stiftleiste_2x10Pm_R2.54
Connections:
- net +3V3: now also R39.1; no longer C19.1, C24.1, C25.1, C26.1, C27.1, C28.1, C29.1, C30.1, C31.1, C32.1, C33.1, C34.1, C35.1, R11.1, R12.1, R13.1, R8.1, R9.1, U3.3 (VDD), xc6slx9_1.103 (VCCO_1), xc6slx9_1.122 (VCCO_0), xc6slx9_1.125 (VCCO_0), xc6slx9_1.135 (VCCO_0), xc6slx9_1.18 (VCCO_3), xc6slx9_1.31 (VCCO_3), xc6slx9_1.4 (VCCO_3), xc6slx9_1.42 (VCCO_2), xc6slx9_1.60 (IO_L13P_M1_2), xc6slx9_1.63 (VCCO_2), xc6slx9_1.69 (IO_L1N_M0_CMPMISO_2), xc6slx9_1.76 (VCCO_1), xc6slx9_1.86 (VCCO_1)
- net Clk_A: now also xc6slx9_1.124 (IO_L37P_GCLK13_0); no longer xc6slx9_1.127 (IO_L36P_GCLK15_0)
- net Clk_B: now also xc6slx9_1.132 (IO_L35P_GCLK17_0); no longer xc6slx9_1.134 (IO_L34P_GCLK19_0)
- net EN_CHA_FILTA: now also xc6slx9_1.126 (IO_L36N_GCLK14_0); no longer xc6slx9_1.10 (IO_L50P_3)
- net EN_CHA_FILTB: now also xc6slx9_1.131 (IO_L35N_GCLK16_0); no longer xc6slx9_1.12 (IO_L49P_3)
- net EN_CHB_FILTA: now also xc6slx9_1.134 (IO_L34P_GCLK19_0); no longer xc6slx9_1.8 (IO_L51P_3)
- net EN_CHB_FILTB: now also xc6slx9_1.133 (IO_L34N_GCLK18_0); no longer xc6slx9_1.6 (IO_L52P_3)
- net Ext_Ref_Clk: now also xc6slx9_1.127 (IO_L36P_GCLK15_0); no longer xc6slx9_1.132 (IO_L35P_GCLK17_0)
- net GND: now also D11.1 (K)
- net LED5: now also xc6slx9_1.51 (IO_L31P_GCLK31_D14_2); no longer xc6slx9_1.35 (IO_L1P_3)
- net LED6: now also xc6slx9_1.50 (IO_L31N_GCLK30_D15_2); no longer xc6slx9_1.34 (IO_L1N_VREF_3)
- net LED7: now also xc6slx9_1.48 (IO_L48P_D7_2); no longer xc6slx9_1.33 (IO_L2P_3)
- net SCL_DAC: now also X1.1
- net SDA_DAC: now also X1.2
- net Int_Ref_Clk: now reaches xc6slx9_1.123 (IO_L37N_GCLK12_0)
- net Int_Ref_Clk: now also G1.8 (CLK)
- net TP10: now reaches xc6slx9_1.11 (IO_L49N_3)
- net TP10: now also X1.12
- net TP8: now reaches xc6slx9_1.14 (IO_L44N_GCLK20_3)
- net TP8: now also X1.10
- net TP7: now reaches xc6slx9_1.15 (IO_L44P_GCLK21_3)
- net TP7: now also X1.9
- net TP6: now reaches xc6slx9_1.16 (IO_L43N_GCLK22_IRDY2_3)
- net TP6: now also X1.8
- net TP5: now reaches xc6slx9_1.17 (IO_L43P_GCLK23_3)
- net TP5: now also X1.7
- net TP4: now reaches xc6slx9_1.21 (IO_L42N_GCLK24_3)
- net TP4: now also X1.6
- net TP3: now reaches xc6slx9_1.22 (IO_L42P_GCLK25_TRDY2_3)
- net TP3: now also X1.5
- net TP2: now reaches xc6slx9_1.23 (IO_L41N_GCLK26_3)
- net TP2: now also X1.4
- net TP1: now reaches xc6slx9_1.24 (IO_L41P_GCLK27_3)
- net TP1: now also X1.3
- net +2V5 renamed +3V3_FPGA
- net +3V3_FPGA: now also C19.1, C24.1, C25.1, C26.1, C27.1, C28.1, C29.1, C30.1, C31.1, C32.1, C33.1, C34.1, C35.1, R11.1, R12.1, R13.1, R8.1, R9.1, U3.3 (VDD), xc6slx9_1.103 (VCCO_1), xc6slx9_1.122 (VCCO_0), xc6slx9_1.125 (VCCO_0), xc6slx9_1.135 (VCCO_0), xc6slx9_1.18 (VCCO_3), xc6slx9_1.31 (VCCO_3), xc6slx9_1.4 (VCCO_3), xc6slx9_1.42 (VCCO_2), xc6slx9_1.60 (IO_L13P_M1_2), xc6slx9_1.63 (VCCO_2), xc6slx9_1.69 (IO_L1N_M0_CMPMISO_2), xc6slx9_1.76 (VCCO_1), xc6slx9_1.86 (VCCO_1)
- removed net Ref_Clk: G1.8 (CLK), xc6slx9_1.124 (IO_L37P_GCLK13_0)
- new net: D11.2 (A), R39.2
- new net TP9: X1.11, xc6slx9_1.12 (IO_L49P_3)
- no-connect marks 77 -> 75
Other:
- moved on the sheet: D1, D10, D2, D3, D4, D5, D6, D7, D8, D9, R14, R15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

Commit message: Update Layout and Schematic [On Change]
Connections:
- net RXD: now also xc6slx9_1.84 (IO_L43N_GCLK4_1); no longer xc6slx9_1.80 (IO_L46N_1)
- net TXD: now also xc6slx9_1.85 (IO_L43P_GCLK5_1); no longer xc6slx9_1.82 (IO_L45N_1)
Changed lines of the file:
@@
 $EndComp
 NoConn ~ 3825 4325
-NoConn ~ 3825 4425
 NoConn ~ 3825 4725
 NoConn ~ 8900 4700
@@
 	1    0    0    -1
 $EndComp
-Text HLabel 4650 4625 2    60   Input ~ 0
+Text HLabel 4650 4450 2    60   Input ~ 0
 RXD
-Text HLabel 4650 4525 2    60   Output ~ 0
+Text HLabel 4650 4350 2    60   Output ~ 0
 TXD
 $Comp
@@
 $EndComp
 Wire Wire Line
-	4650 4525 3825 4525
-Wire Wire Line
 	6600 3300 6600 3500
 Wire Wire Line
@@
 Wire Wire Line
 	6325 4950 6250 4950
-Wire Wire Line
-	3825 4625 4650 4625
 $Comp
 L LED D3
@@
 NoConn ~ 6250 4450
 NoConn ~ 3825 4275
-NoConn ~ 3825 4375
 NoConn ~ 3825 4575
 $Comp
@@
 Wire Wire Line
 	3800 6750 3800 6725
+NoConn ~ 3825 4625
+NoConn ~ 3825 4525
+Wire Wire Line
+	4650 4350 4525 4350
+Wire Wire Line
+	4525 4350 4525 4375
+Wire Wire Line
+	4525 4375 3825 4375
+Wire Wire Line
+	3825 4425 4525 4425
+Wire Wire Line
+	4525 4425 4525 4450
+Wire Wire Line
+	4525 4450 4650 4450
 $EndSCHEMATC
