File: kicad/FPGA.sch (KiCad schematic (older format))
At the start: 56 parts, among them U3 MCP4725, X1 Stiftleiste_2x10Pm_R2.54

Commit message: Layout changes [in progress]
Parts:
- removed D10, D3, D4, D9: LED, Footprints_LJ:Mini_TopLed_SMD, symbol LED
- removed R16, R17, R22, R23: 680R, Resistors_SMD:R_0603_HandSoldering, symbol R
- added C?: 1u, symbol C
- added R?: 1k, symbol R
Connections:
- net +3V3_FPGA: no longer xc6slx9_1.60 (IO_L13P_M1_2)
- net GND: now also xc6slx9_1.60 (IO_L13P_M1_2), C?.2
- net LED0: now also R18.1
- net LED1: now also R19.1
- net LED2: now also R20.1; no longer R18.1
- net LED3: now also R21.1; no longer R19.1
- net at U3.1 (VOUT): now also R?.1; no longer G1.1 (CTR_V)
- net LED4: no longer names the net of xc6slx9_1.55 (IO_L30N_GCLK0_USERCCLK_2)
- net LED4: no longer R20.1
- net LED5: no longer names the net of xc6slx9_1.51 (IO_L31P_GCLK31_D14_2)
- net LED5: no longer R21.1
- net LED6: no longer names the net of xc6slx9_1.50 (IO_L31N_GCLK30_D15_2)
- net LED7: no longer names the net of xc6slx9_1.48 (IO_L48P_D7_2)
- new net: C?.1, G1.1 (CTR_V), R?.2
- no-connect marks 75 -> 79
Other:
- moved on the sheet: D5, D6, D7, D8, R18, R19, R20, R21, R9

Commit message: Layout changes [In progress]
Parts:
- C8: renamed from C?; footprint (none) -> Capacitors_SMD:C_0603_HandSoldering
- R16: renamed from R?; footprint (none) -> Resistors_SMD:R_0603_HandSoldering
Connections:
- net +3V3: now also C19.1, R8.1, R9.1, U3.3 (VDD)
- net +3V3_FPGA: no longer C19.1, R8.1, R9.1, U3.3 (VDD)
Changed lines of the file:
@@
 	3775 7125 3775 7100
 $Comp
-L +3V3_FPGA #PWR068
+L +3V3_FPGA #PWR060
 U 1 1 5971EC0E
 P 9100 4725
-F 0 "#PWR068" H 9100 4575 50  0001 C CNN
+F 0 "#PWR060" H 9100 4575 50  0001 C CNN
 F 1 "+3V3_FPGA" H 9100 4865 50  0000 C CNN
 F 2 "" H 9100 4725 50  0001 C CNN
@@
 $EndComp
 $Comp
-L +3V3_FPGA #PWR069
+L +3V3_FPGA #PWR061
 U 1 1 5971EC9A
 P 1575 4875
-F 0 "#PWR069" H 1575 4725 50  0001 C CNN
+F 0 "#PWR061" H 1575 4725 50  0001 C CNN
 F 1 "+3V3_FPGA" H 1575 5015 50  0000 C CNN
 F 2 "" H 1575 4875 50  0001 C CNN
@@
 $EndComp
 $Comp
-L +3V3_FPGA #PWR070
+L +3V3_FPGA #PWR062
 U 1 1 5971F302
 P 7400 4400
-F 0 "#PWR070" H 7400 4250 50  0001 C CNN
+F 0 "#PWR062" H 7400 4250 50  0001 C CNN
 F 1 "+3V3_FPGA" H 7400 4540 50  0000 C CNN
 F 2 "" H 7400 4400 50  0001 C CNN
@@
 $EndComp
 $Comp
-L +3V3_FPGA #PWR072
+L +3V3_FPGA #PWR063
 U 1 1 5971F636
 P 4700 7125
-F 0 "#PWR072" H 4700 6975 50  0001 C CNN
+F 0 "#PWR063" H 4700 6975 50  0001 C CNN
 F 1 "+3V3_FPGA" H 4700 7265 50  0000 C CNN
 F 2 "" H 4700 7125 50  0001 C CNN
@@
 $EndComp
 $Comp
-L +3V3_FPGA #PWR073
+L +3V3_FPGA #PWR064
 U 1 1 5971F6C2
 P 5600 7125
-F 0 "#PWR073" H 5600 6975 50  0001 C CNN
+F 0 "#PWR064" H 5600 6975 50  0001 C CNN
 F 1 "+3V3_FPGA" H 5600 7265 50  0000 C CNN
 F 2 "" H 5600 7125 50  0001 C CNN
@@
 $EndComp
 $Comp
-L +3V3_FPGA #PWR074
+L +3V3_FPGA #PWR065
 U 1 1 5971F74E
 P 6650 7125
-F 0 "#PWR074" H 6650 6975 50  0001 C CNN
+F 0 "#PWR065" H 6650 6975 50  0001 C CNN
 F 1 "+3V3_FPGA" H 6650 7265 50  0000 C CNN
 F 2 "" H 6650 7125 50  0001 C CNN
@@
 $EndComp
 $Comp
-L +3V3_FPGA #PWR075
+L +3V3_FPGA #PWR066
 U 1 1 5971F9F6
 P 7475 3000
-F 0 "#PWR075" H 7475 2850 50  0001 C CNN
+F 0 "#PWR066" H 7475 2850 50  0001 C CNN
 F 1 "+3V3_FPGA" H 7475 3140 50  0000 C CNN
 F 2 "" H 7475 3000 50  0001 C CNN
@@
 $EndComp
 $Comp
-L +3V3_FPGA #PWR076
+L +3V3_FPGA #PWR067
 U 1 1 5971FA82
 P 6600 3000
-F 0 "#PWR076" H 6600 2850 50  0001 C CNN
+F 0 "#PWR067" H 6600 2850 50  0001 C CNN
 F 1 "+3V3_FPGA" H 6600 3140 50  0000 C CNN
 F 2 "" H 6600 3000 50  0001 C CNN
@@
 $EndComp
 $Comp
-L +3V3_FPGA #PWR077
-U 1 1 5971FD2A
-P 4300 1100
-F 0 "#PWR077" H 4300 950 50  0001 C CNN
-F 1 "+3V3_FPGA" H 4300 1240 50  0000 C CNN
-F 2 "" H 4300 1100 50  0001 C CNN
-F 3 "" H 4300 1100 50  0001 C CNN
-	1    4300 1100
-	1    0    0    -1
-$EndComp
-$Comp
-L +3V3_FPGA #PWR078
+L +3V3_FPGA #PWR069
 U 1 1 5972013B
 P 10500 900
-F 0 "#PWR078" H 10500 750 50  0001 C CNN
+F 0 "#PWR069" H 10500 750 50  0001 C CNN
 F 1 "+3V3_FPGA" H 10500 1040 50  0000 C CNN
 F 2 "" H 10500 900 50  0001 C CNN
@@
 NoConn ~ 1375 4800
 $Comp
-L +3V3_FPGA #PWR079
-U 1 1 5973F5C6
-P 4700 1300
-F 0 "#PWR079" H 4700 1150 50  0001 C CNN
-F 1 "+3V3_FPGA" H 4700 1440 50  0000 C CNN
-F 2 "" H 4700 1300 50  0001 C CNN
-F 3 "" H 4700 1300 50  0001 C CNN
-	1    4700 1300
-	1    0    0    -1
-$EndComp
-$Comp
-L +3V3_FPGA #PWR080
+L +3V3_FPGA #PWR071
 U 1 1 5973FE95
 P 6350 3000
-F 0 "#PWR080" H 6350 2850 50  0001 C CNN
+F 0 "#PWR071" H 6350 2850 50  0001 C CNN
 F 1 "+3V3_FPGA" H 6350 3140 50  0000 C CNN
 F 2 "" H 6350 3000 50  0001 C CNN
@@
 $EndComp
 $Comp
-L GND #PWR081
+L GND #PWR072
 U 1 1 5974536A
 P 725 6750
-F 0 "#PWR081" H 725 6500 50  0001 C CNN
+F 0 "#PWR072" H 725 6500 50  0001 C CNN
 F 1 "GND" H 725 6600 50  0000 C CNN
 F 2 "" H 725 6750 50  0001 C CNN
@@
 $EndComp
 $Comp
-L +3V3 #PWR082
+L +3V3 #PWR073
 U 1 1 597454BF
 P 725 6100
-F 0 "#PWR082" H 725 5950 50  0001 C CNN
+F 0 "#PWR073" H 725 5950 50  0001 C CNN
 F 1 "+3V3" H 725 6240 50  0000 C CNN
 F 2 "" H 725 6100 50  0001 C CNN
@@
 Connection ~ 9100 4750
 $Comp
-L +3V3_FPGA #PWR083
+L +3V3_FPGA #PWR074
 U 1 1 59756293
 P 3925 4850
-F 0 "#PWR083" H 3925 4700 50  0001 C CNN
+F 0 "#PWR074" H 3925 4700 50  0001 C CNN
 F 1 "+3V3_FPGA" H 3925 4990 50  0000 C CNN
 F 2 "" H 3925 4850 50  0001 C CNN
@@
 	2575 6100 2575 6125
 $Comp
-L GND #PWR065
+L GND #PWR075
 U 1 1 59710CC9
 P 2575 6750
-F 0 "#PWR065" H 2575 6500 50  0001 C CNN
+F 0 "#PWR075" H 2575 6500 50  0001 C CNN
 F 1 "GND" H 2575 6600 50  0000 C CNN
 F 2 "" H 2575 6750 50  0001 C CNN
@@
 	2300 6100 2300 6125
 $Comp
-L GND #PWR064
+L GND #PWR076
 U 1 1 59710CAE
 P 2300 6750
-F 0 "#PWR064" H 2300 6500 50  0001 C CNN
+F 0 "#PWR076" H 2300 6500 50  0001 C CNN
 F 1 "GND" H 2300 6600 50  0000 C CNN
 F 2 "" H 2300 6750 50  0001 C CNN
@@
 	2000 6100 2000 6125
 $Comp
-L GND #PWR063
+L GND #PWR077
 U 1 1 59710C93
 P 2000 6750
-F 0 "#PWR063" H 2000 6500 50  0001 C CNN
+F 0 "#PWR077" H 2000 6500 50  0001 C CNN
 F 1 "GND" H 2000 6600 50  0000 C CNN
 F 2 "" H 2000 6750 50  0001 C CNN
@@
 	1700 6100 1700 6125
 $Comp
-L GND #PWR062
+L GND #PWR078
 U 1 1 5971084E
 P 1700 6750
-F 0 "#PWR062" H 1700 6500 50  0001 C CNN
+F 0 "#PWR078" H 1700 6500 50  0001 C CNN
 F 1 "GND" H 1700 6600 50  0000 C CNN
 F 2 "" H 1700 6750 50  0001 C CNN
@@
 LED0
 $Comp
-L R R?
+L R R16
 U 1 1 59BAADBE
 P 3250 2450
-F 0 "R?" V 3330 2450 50  0000 C CNN
+F 0 "R16" V 3330 2450 50  0000 C CNN
 F 1 "1k" V 3250 2450 50  0000 C CNN
-F 2 "" V 3180 2450 50  0001 C CNN
+F 2 "Resistors_SMD:R_0603_HandSoldering" V 3180 2450 50  0001 C CNN
 F 3 "" H 3250 2450 50  0001 C CNN
 	1    3250 2450
@@
 $EndComp
 $Comp
-L C C?
+L C C8
 U 1 1 59BAAF37
 P 2900 2600
-F 0 "C?" H 2925 2700 50  0000 L CNN
+F 0 "C8" H 2925 2700 50  0000 L CNN
 F 1 "1u" H 2925 2500 50  0000 L CNN
-F 2 "" H 2938 2450 50  0001 C CNN
+F 2 "Capacitors_SMD:C_0603_HandSoldering" H 2938 2450 50  0001 C CNN
 F 3 "" H 2900 2600 50  0001 C CNN
 	1    2900 2600
@@
 	7050 2450 3400 2450
 $Comp
-L GND #PWR?
+L GND #PWR079
 U 1 1 59BAB3E9
 P 2900 2750
-F 0 "#PWR?" H 2900 2500 50  0001 C CNN
+F 0 "#PWR079" H 2900 2500 50  0001 C CNN
 F 1 "GND" H 2900 2600 50  0000 C CNN
 F 2 "" H 2900 2750 50  0001 C CNN
@@
 	6300 3950 6300 5025
 $Comp
-L GND #PWR?
+L GND #PWR080
 U 1 1 59BAF83E
 P 6300 5025
-F 0 "#PWR?" H 6300 4775 50  0001 C CNN
+F 0 "#PWR080" H 6300 4775 50  0001 C CNN
 F 1 "GND" H 6300 4875 50  0000 C CNN
 F 2 "" H 6300 5025 50  0001 C CNN
@@
 	4225 4225 4450 4225
 $Comp
-L +3V3_FPGA #PWR?
+L +3V3_FPGA #PWR081
 U 1 1 59BC3F1E
 P 3375 7125
-F 0 "#PWR?" H 3375 6975 50  0001 C CNN
+F 0 "#PWR081" H 3375 6975 50  0001 C CNN
 F 1 "+3V3_FPGA" H 3375 7265 50  0000 C CNN
 F 2 "" H 3375 7125 50  0001 C CNN
@@
 Wire Wire Line
 	4400 1200 4400 1275
+$Comp
+L +3.3V #PWR?
+U 1 1 59C164D1
+P 4300 1100
+F 0 "#PWR?" H 4300 950 50  0001 C CNN
+F 1 "+3.3V" H 4300 1240 50  0000 C CNN
+F 2 "" H 4300 1100 50  0001 C CNN
+F 3 "" H 4300 1100 50  0001 C CNN
+	1    4300 1100
+	1    0    0    -1
+$EndComp
+$Comp
+L +3.3V #PWR?
+U 1 1 59C16555
+P 4700 1300
+F 0 "#PWR?" H 4700 1150 50  0001 C CNN
+F 1 "+3.3V" H 4700 1440 50  0000 C CNN
+F 2 "" H 4700 1300 50  0001 C CNN
+F 3 "" H 4700 1300 50  0001 C CNN
+	1    4700 1300
+	1    0    0    -1
+$EndComp
 $EndSCHEMATC

Commit message: Rework hardware schematic [in progress]
Parts:
- added U11: tx176, Footprints_LJ:tx176, symbol tx176
Connections:
- net +3V3: now also U11.9 (VCC)
- net Clk_A: now also xc6slx9_1.14 (IO_L44N_GCLK20_3); no longer xc6slx9_1.124 (IO_L37P_GCLK13_0)
- net Clk_B: now also xc6slx9_1.21 (IO_L42N_GCLK24_3); no longer xc6slx9_1.132 (IO_L35P_GCLK17_0)
- net EN_CHA_FILTA: now also xc6slx9_1.10 (IO_L50P_3); no longer xc6slx9_1.126 (IO_L36N_GCLK14_0)
- net EN_CHA_FILTB: now also xc6slx9_1.8 (IO_L51P_3); no longer xc6slx9_1.131 (IO_L35N_GCLK16_0)
- net EN_CHB_FILTA: now also xc6slx9_1.34 (IO_L1N_VREF_3); no longer xc6slx9_1.134 (IO_L34P_GCLK19_0)
- net EN_CHB_FILTB: now also xc6slx9_1.32 (IO_L2N_3); no longer xc6slx9_1.133 (IO_L34N_GCLK18_0)
- net Ext_Ref_Clk: now also xc6slx9_1.16 (IO_L43N_GCLK22_IRDY2_3); no longer xc6slx9_1.127 (IO_L36P_GCLK15_0)
- net GND: now also U11.4 (GND)
- net Int_Ref_Clk: now also xc6slx9_1.50 (IO_L31N_GCLK30_D15_2), U11.5 (OUT~); no longer xc6slx9_1.123 (IO_L37N_GCLK12_0)
- net LED0: now also xc6slx9_1.62 (IO_L12P_D1_MISO2_2); no longer xc6slx9_1.59 (IO_L13N_D10_2)
- net LED1: now also xc6slx9_1.59 (IO_L13N_D10_2); no longer xc6slx9_1.58 (IO_L14P_D11_2)
- net LED2: now also xc6slx9_1.56 (IO_L30P_GCLK1_D13_2); no longer xc6slx9_1.57 (IO_L14N_D12_2)
- net LED3: now also xc6slx9_1.46 (IO_L49P_D3_2); no longer xc6slx9_1.56 (IO_L30P_GCLK1_D13_2)
- net RXD: now also xc6slx9_1.87 (IO_L42N_GCLK6_TRDY1_1); no longer xc6slx9_1.84 (IO_L43N_GCLK4_1)
- net SCL_DAC: now also xc6slx9_1.23 (IO_L41N_GCLK26_3); no longer xc6slx9_1.93 (IO_L41P_GCLK9_IRDY1_1)
- net SDA_DAC: now also xc6slx9_1.24 (IO_L41P_GCLK27_3); no longer xc6slx9_1.94 (IO_L40N_GCLK10_1)
- net TP1: now also xc6slx9_1.134 (IO_L34P_GCLK19_0); no longer xc6slx9_1.24 (IO_L41P_GCLK27_3)
- net TP10: now also xc6slx9_1.120 (IO_L62N_VREF_0); no longer xc6slx9_1.11 (IO_L49N_3)
- net TP2: now also xc6slx9_1.133 (IO_L34N_GCLK18_0); no longer xc6slx9_1.23 (IO_L41N_GCLK26_3)
- net TP3: now also xc6slx9_1.132 (IO_L35P_GCLK17_0); no longer xc6slx9_1.22 (IO_L42P_GCLK25_TRDY2_3)
- net TP4: now also xc6slx9_1.131 (IO_L35N_GCLK16_0); no longer xc6slx9_1.21 (IO_L42N_GCLK24_3)
- net TP5: now also xc6slx9_1.127 (IO_L36P_GCLK15_0); no longer xc6slx9_1.17 (IO_L43P_GCLK23_3)
- net TP6: now also xc6slx9_1.126 (IO_L36N_GCLK14_0); no longer xc6slx9_1.16 (IO_L43N_GCLK22_IRDY2_3)
- net TP7: now also xc6slx9_1.124 (IO_L37P_GCLK13_0); no longer xc6slx9_1.15 (IO_L44P_GCLK21_3)
- net TP8: now also xc6slx9_1.123 (IO_L37N_GCLK12_0); no longer xc6slx9_1.14 (IO_L44N_GCLK20_3)
- net TP9: now also xc6slx9_1.121 (IO_L62P_0); no longer xc6slx9_1.12 (IO_L49P_3)
- net TXD: now also xc6slx9_1.88 (IO_L42P_GCLK7_1); no longer xc6slx9_1.85 (IO_L43P_GCLK5_1)
- net at C8.1, G1.1 (CTR_V), R16.2: now also U11.10 (CV)
Other:
- moved on the sheet: C23, C8, G1, R13, R16

Commit message: Layout changes [in progress]
Parts:
- removed D5, D6, D7, D8: LED, Footprints_LJ:Mini_TopLed_SMD, symbol LED
- removed R18, R19, R20, R21: 680R, Resistors_SMD:R_0603_HandSoldering, symbol R
- R12: footprint Resistors_SMD:R_0612 -> Resistors_SMD:R_0603_HandSoldering
Connections:
- net LED0: no longer names the net of xc6slx9_1.62 (IO_L12P_D1_MISO2_2)
- net LED1: no longer names the net of xc6slx9_1.59 (IO_L13N_D10_2)
- net LED2: no longer names the net of xc6slx9_1.56 (IO_L30P_GCLK1_D13_2)
- net LED3: no longer names the net of xc6slx9_1.46 (IO_L49P_D3_2)
- no-connect marks 79 -> 78
Changed lines of the file:
@@
 F 0 "R12" V 7555 3150 50  0000 C CNN
 F 1 "4.7k" V 7475 3150 50  0000 C CNN
-F 2 "Resistors_SMD:R_0612" V 7405 3150 50  0001 C CNN
+F 2 "Resistors_SMD:R_0603_HandSoldering" V 7405 3150 50  0001 C CNN
 F 3 "" H 7475 3150 50  0001 C CNN
 	1    7475 3150
@@
 	1    0    0    -1
 $EndComp
-Text GLabel 6850 3850 2    60   Output ~ 0
-LED0
-Text GLabel 6850 4000 2    60   Output ~ 0
-LED1
 $Comp
 L AOCJY1-100MHz G1
@@
 NoConn ~ 3825 4625
 NoConn ~ 3825 4525
-Text GLabel 6850 4450 2    60   Output ~ 0
-LED3
-Text GLabel 6850 4150 2    60   Output ~ 0
-LED2
-$Comp
-L R R21
-U 1 1 59710CD0
-P 2575 6275
-F 0 "R21" V 2655 6275 50  0000 C CNN
-F 1 "680R" V 2575 6275 50  0000 C CNN
-F 2 "Resistors_SMD:R_0603_HandSoldering" V 2505 6275 50  0001 C CNN
-F 3 "" H 2575 6275 50  0001 C CNN
-	1    2575 6275
-	1    0    0    -1
-$EndComp
-$Comp
-L GND #PWR072
-U 1 1 59710CC9
-P 2575 6750
-F 0 "#PWR072" H 2575 6500 50  0001 C CNN
-F 1 "GND" H 2575 6600 50  0000 C CNN
-F 2 "" H 2575 6750 50  0001 C CNN
-F 3 "" H 2575 6750 50  0001 C CNN
-	1    2575 6750
-	1    0    0    -1
-$EndComp
-$Comp
-L LED D8
-U 1 1 59710CC2
-P 2575 6575
-F 0 "D8" H 2575 6675 50  0000 C CNN
-F 1 "LED" H 2575 6475 50  0000 C CNN
-F 2 "Footprints_LJ:Mini_TopLed_SMD" H 2575 6575 50  0001 C CNN
-F 3 "" H 2575 6575 50  0001 C CNN
-	1    2575 6575
-	0    -1   -1   0
-$EndComp
-$Comp
-L R R20
-U 1 1 59710CB5
-P 2300 6275
-F 0 "R20" V 2380 6275 50  0000 C CNN
-F 1 "680R" V 2300 6275 50  0000 C CNN
-F 2 "Resistors_SMD:R_0603_HandSoldering" V 2230 6275 50  0001 C CNN
-F 3 "" H 2300 6275 50  0001 C CNN
-	1    2300 6275
-	1    0    0    -1
-$EndComp
-$Comp
-L GND #PWR073
-U 1 1 59710CAE
-P 2300 6750
-F 0 "#PWR073" H 2300 6500 50  0001 C CNN
-F 1 "GND" H 2300 6600 50  0000 C CNN
-F 2 "" H 2300 6750 50  0001 C CNN
-F 3 "" H 2300 6750 50  0001 C CNN
-	1    2300 6750
-	1    0    0    -1
-$EndComp
-$Comp
-L LED D7
-U 1 1 59710CA7
-P 2300 6575
-F 0 "D7" H 2300 6675 50  0000 C CNN
-F 1 "LED" H 2300 6475 50  0000 C CNN
-F 2 "Footprints_LJ:Mini_TopLed_SMD" H 2300 6575 50  0001 C CNN
-F 3 "" H 2300 6575 50  0001 C CNN
-	1    2300 6575
-	0    -1   -1   0
-$EndComp
-$Comp
-L R R19
-U 1 1 59710C9A
-P 2000 6275
-F 0 "R19" V 2080 6275 50  0000 C CNN
-F 1 "680R" V 2000 6275 50  0000 C CNN
-F 2 "Resistors_SMD:R_0603_HandSoldering" V 1930 6275 50  0001 C CNN
-F 3 "" H 2000 6275 50  0001 C CNN
-	1    2000 6275
-	1    0    0    -1
-$EndComp
-$Comp
-L GND #PWR074
-U 1 1 59710C93
-P 2000 6750
-F 0 "#PWR074" H 2000 6500 50  0001 C CNN
-F 1 "GND" H 2000 6600 50  0000 C CNN
-F 2 "" H 2000 6750 50  0001 C CNN
-F 3 "" H 2000 6750 50  0001 C CNN
-	1    2000 6750
-	1    0    0    -1
-$EndComp
-$Comp
-L LED D6
-U 1 1 59710C8C
-P 2000 6575
-F 0 "D6" H 2000 6675 50  0000 C CNN
-F 1 "LED" H 2000 6475 50  0000 C CNN
-F 2 "Footprints_LJ:Mini_TopLed_SMD" H 2000 6575 50  0001 C CNN
-F 3 "" H 2000 6575 50  0001 C CNN
-	1    2000 6575
-	0    -1   -1   0
-$EndComp
-$Comp
-L R R18
-U 1 1 59710855
-P 1700 6275
-F 0 "R18" V 1780 6275 50  0000 C CNN
-F 1 "680R" V 1700 6275 50  0000 C CNN
-F 2 "Resistors_SMD:R_0603_HandSoldering" V 1630 6275 50  0001 C CNN
-F 3 "" H 1700 6275 50  0001 C CNN
-	1    1700 6275
-	1    0    0    -1
-$EndComp
-$Comp
-L GND #PWR075
-U 1 1 5971084E
-P 1700 6750
-F 0 "#PWR075" H 1700 6500 50  0001 C CNN
-F 1 "GND" H 1700 6600 50  0000 C CNN
-F 2 "" H 1700 6750 50  0001 C CNN
-F 3 "" H 1700 6750 50  0001 C CNN
-	1    1700 6750
-	1    0    0    -1
-$EndComp
-$Comp
-L LED D5
-U 1 1 59710847
-P 1700 6575
-F 0 "D5" H 1700 6675 50  0000 C CNN
-F 1 "LED" H 1700 6475 50  0000 C CNN
-F 2 "Footprints_LJ:Mini_TopLed_SMD" H 1700 6575 50  0001 C CNN
-F 3 "" H 1700 6575 50  0001 C CNN
-	1    1700 6575
-	0    -1   -1   0
-$EndComp
-Text GLabel 2575 6100 1    60   Input ~ 0
-LED3
-Text GLabel 2300 6100 1    60   Input ~ 0
-LED2
-Text GLabel 2000 6100 1    60   Input ~ 0
-LED1
-Text GLabel 1700 6100 1    60   Input ~ 0
-LED0
 $Comp
 L R R16
@@
 Connection ~ 6600 3375
 Wire Wire Line
-	6250 4000 6850 4000
-Wire Wire Line
 	4200 1275 4200 1200
 Wire Wire Line
@@
 Wire Wire Line
 	4525 4350 4650 4350
-Wire Wire Line
-	2575 6750 2575 6725
-Wire Wire Line
-	2300 6750 2300 6725
-Wire Wire Line
-	2000 6750 2000 6725
-Wire Wire Line
-	1700 6750 1700 6725
-Wire Wire Line
-	2575 6100 2575 6125
-Wire Wire Line
-	2300 6100 2300 6125
-Wire Wire Line
-	2000 6100 2000 6125
-Wire Wire Line
-	1700 6100 1700 6125
 Connection ~ 4975 2500
 Wire Wire Line
@@
 NoConn ~ 6250 4250
 NoConn ~ 6250 4200
-NoConn ~ 6250 3900
 NoConn ~ 6250 3800
 NoConn ~ 6250 3750
@@
 NoConn ~ 8900 3750
 NoConn ~ 8900 3800
-Wire Wire Line
-	6850 3850 6250 3850
 NoConn ~ 6250 4050
 NoConn ~ 6250 4100
-Wire Wire Line
-	6250 4150 6850 4150
 NoConn ~ 6250 4350
 NoConn ~ 6250 4500
 NoConn ~ 6250 4550
 Wire Wire Line
-	6250 4450 6850 4450
-Wire Wire Line
 	6850 4300 6250 4300

Commit message: Reworked schematic and layout [to review]
Connections:
- net EN_CHA_FILTB is gone; now on net TP9: xc6slx9_1.8 (IO_L51P_3)
- net Clk_A: now also xc6slx9_1.134 (IO_L34P_GCLK19_0); no longer xc6slx9_1.14 (IO_L44N_GCLK20_3)
- net Clk_B: now also xc6slx9_1.14 (IO_L44N_GCLK20_3); no longer xc6slx9_1.21 (IO_L42N_GCLK24_3)
- net Ext_Ref_Clk: now also xc6slx9_1.24 (IO_L41P_GCLK27_3); no longer xc6slx9_1.16 (IO_L43N_GCLK22_IRDY2_3)
- net Int_Ref_Clk: now also xc6slx9_1.56 (IO_L30P_GCLK1_D13_2); no longer xc6slx9_1.50 (IO_L31N_GCLK30_D15_2)
- net SCL_DAC: now also X1.11, xc6slx9_1.15 (IO_L44P_GCLK21_3); no longer X1.1, xc6slx9_1.23 (IO_L41N_GCLK26_3)
- net SDA_DAC: now also X1.12, xc6slx9_1.16 (IO_L43N_GCLK22_IRDY2_3); no longer X1.2, xc6slx9_1.24 (IO_L41P_GCLK27_3)
- net TP1: now also X1.1, xc6slx9_1.137 (IO_L4N_0); no longer X1.3, xc6slx9_1.134 (IO_L34P_GCLK19_0)
- net TP10: now also X1.10, xc6slx9_1.9 (IO_L50N_3); no longer X1.12, xc6slx9_1.120 (IO_L62N_VREF_0)
- net TP2: now also X1.2, xc6slx9_1.138 (IO_L4P_0); no longer X1.4, xc6slx9_1.133 (IO_L34N_GCLK18_0)
- net TP3: now also X1.3, xc6slx9_1.139 (IO_L3N_0); no longer X1.5, xc6slx9_1.132 (IO_L35P_GCLK17_0)
- net TP4: now also X1.4, xc6slx9_1.140 (IO_L3P_0); no longer X1.6, xc6slx9_1.131 (IO_L35N_GCLK16_0)
- net TP5: now also X1.5, xc6slx9_1.141 (IO_L2N_0); no longer X1.7, xc6slx9_1.127 (IO_L36P_GCLK15_0)
- net TP6: now also X1.6, xc6slx9_1.5 (IO_L52N_3); no longer X1.8, xc6slx9_1.126 (IO_L36N_GCLK14_0)
- net TP7: now also X1.7, xc6slx9_1.6 (IO_L52P_3); no longer X1.9, xc6slx9_1.124 (IO_L37P_GCLK13_0)
- net TP8: now also X1.8, xc6slx9_1.7 (IO_L51N_3); no longer X1.10, xc6slx9_1.123 (IO_L37N_GCLK12_0)
- net TP9: now also X1.9; no longer X1.11, xc6slx9_1.121 (IO_L62P_0)
- net EN_EXTREF_FILTB: now reaches xc6slx9_1.17 (IO_L43P_GCLK23_3)
- net EN_EXTREF_FILTA: now reaches xc6slx9_1.22 (IO_L42P_GCLK25_TRDY2_3)
- net EN_CHA_FILTA: no longer names the net of xc6slx9_1.10 (IO_L50P_3)
- net EN_CHB_FILTA: no longer names the net of xc6slx9_1.34 (IO_L1N_VREF_3)
- net EN_CHB_FILTB: no longer names the net of xc6slx9_1.32 (IO_L2N_3)
- no-connect marks 78 -> 85

Commit message: some small schematic and layout changes [completed]
Parts:
- removed R12, R13: 4.7k, Resistors_SMD:R_0603_HandSoldering, symbol R
- added C_I2C_1, C_I2C_2, C_JTAG_1, C_JTAG_2, C_RS2232_1, C_RS2232_2, C_TP_1, C_TP_2: 1u, Capacitors_SMD:C_0603_HandSoldering, symbol C
Connections:
- net +1.2V: now also C_JTAG_1.1, C_JTAG_2.1
- net +3V3: now also C_I2C_1.2, C_I2C_2.2, C_JTAG_1.2, C_JTAG_2.2, C_RS2232_1.2, C_RS2232_2.2, C_TP_1.2, C_TP_2.2
- net +3V3_FPGA: now also C_I2C_1.1, C_I2C_2.1, C_RS2232_1.1, C_RS2232_2.1, C_TP_1.1, C_TP_2.1
- net at xc6slx9_1.39 (IO_L65P_INIT_B_2): no longer xc6slx9_1.37 (PROGRAM_B_2)
- new net ~RESET: xc6slx9_1.37 (PROGRAM_B_2)
- no-connect marks 85 -> 87
Other:
- note added: "PowerPlaneCrossing I2C\n\n"
- note added: "PowerPlaneCrossing JTAG\n\n"
- note added: "PowerPlaneCrossing RS2232\n\n\n"
- note added: "PowerPlaneCrossing TPs\n"
- moved on the sheet: C19, C23, C24, C25, C26, C27, C28, C29, C30, C31, C32, C33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
