File: kicad/FPGA.sch (KiCad schematic (older format))
At the start: 49 parts, among them U11 tx176, U3 MCP4725, X1 Stiftleiste_2x10Pm_R2.54

Commit message: Small schematic and layout changes
Connections:
- net ~RESET is gone; now on net +3V3_FPGA: xc6slx9_1.37 (PROGRAM_B_2)
- net +3V3_FPGA: now also xc6slx9_1.65 (IO_L3P_D0_DIN_MISO_MISO1_2)
- net DIV_SW1: now reaches xc6slx9_1.132 (IO_L35P_GCLK17_0)
- net DIV_SW2: now reaches xc6slx9_1.143 (IO_L1N_VREF_0)
- no-connect marks 87 -> 84
Other:
- moved on the sheet: C_I2C_2, R11

Commit message: clean up in layout & add exports (assembly drawings)
Parts:
- C11, C12, C13, C14, C15, C16, C17, C18, C19, C20, C21, C22, C23, C24, C25, C26, C27, C28, C29, C30, C31, C32, C33, C34, C35, C8, C_I2C_1, C_I2C_2, C_JTAG_1, C_JTAG_2, C_RS2232_1, C_RS2232_2, C_TP_1, C_TP_2: footprint Capacitors_SMD:C_0603_HandSoldering -> Footprints_LJ:Cap_0603_HandSoldering_1
Changed lines of the file:
@@
 F 0 "C23" H 1125 2075 50  0000 L CNN
 F 1 "100n" H 1125 1875 50  0000 L CNN
-F 2 "Capacitors_SMD:C_0603_HandSoldering" H 1138 1825 50  0001 C CNN
+F 2 "Footprints_LJ:Cap_0603_HandSoldering_1" H 1138 1825 50  0001 C CNN
 F 3 "" H 1100 1975 50  0001 C CNN
 	1    1100 1975
@@
 F 0 "C19" H 6150 1300 50  0000 L CNN
 F 1 "100n" H 6150 1100 50  0000 L CNN
-F 2 "Capacitors_SMD:C_0603_HandSoldering" H 6163 1050 50  0001 C CNN
+F 2 "Footprints_LJ:Cap_0603_HandSoldering_1" H 6163 1050 50  0001 C CNN
 F 3 "" H 6125 1200 50  0001 C CNN
 	1    6125 1200
@@
 F 0 "C11" H 9125 1225 50  0000 L CNN
 F 1 "4.7u" H 9125 1025 50  0000 L CNN
-F 2 "Capacitors_SMD:C_0603_HandSoldering" H 9138 975 50  0001 C CNN
+F 2 "Footprints_LJ:Cap_0603_HandSoldering_1" H 9138 975 50  0001 C CNN
 F 3 "" H 9100 1125 50  0001 C CNN
 	1    9100 1125
@@
 F 0 "C24" H 9725 5500 50  0000 L CNN
 F 1 "4.7u" H 9725 5300 50  0000 L CNN
-F 2 "Capacitors_SMD:C_0603_HandSoldering" H 9738 5250 50  0001 C CNN
+F 2 "Footprints_LJ:Cap_0603_HandSoldering_1" H 9738 5250 50  0001 C CNN
 F 3 "" H 9700 5400 50  0001 C CNN
 	1    9700 5400
@@
 F 0 "C25" H 9925 5500 50  0000 L CNN
 F 1 "0.47u" H 9925 5300 50  0000 L CNN
-F 2 "Capacitors_SMD:C_0603_HandSoldering" H 9938 5250 50  0001 C CNN
+F 2 "Footprints_LJ:Cap_0603_HandSoldering_1" H 9938 5250 50  0001 C CNN
 F 3 "" H 9900 5400 50  0001 C CNN
 	1    9900 5400
@@
 F 0 "C27" H 9725 6225 50  0000 L CNN
 F 1 "4.7u" H 9725 6025 50  0000 L CNN
-F 2 "Capacitors_SMD:C_0603_HandSoldering" H 9738 5975 50  0001 C CNN
+F 2 "Footprints_LJ:Cap_0603_HandSoldering_1" H 9738 5975 50  0001 C CNN
 F 3 "" H 9700 6125 50  0001 C CNN
 	1    9700 6125
@@
 F 0 "C28" H 9925 6225 50  0000 L CNN
 F 1 "0.47u" H 9925 6025 50  0000 L CNN
-F 2 "Capacitors_SMD:C_0603_HandSoldering" H 9938 5975 50  0001 C CNN
+F 2 "Footprints_LJ:Cap_0603_HandSoldering_1" H 9938 5975 50  0001 C CNN
 F 3 "" H 9900 6125 50  0001 C CNN
 	1    9900 6125
@@
 F 0 "C29" H 10125 6225 50  0000 L CNN
 F 1 "0.47u" H 10125 6025 50  0000 L CNN
-F 2 "Capacitors_SMD:C_0603_HandSoldering" H 10138 5975 50  0001 C CNN
+F 2 "Footprints_LJ:Cap_0603_HandSoldering_1" H 10138 5975 50  0001 C CNN
 F 3 "" H 10100 6125 50  0001 C CNN
 	1    10100 6125
@@
 F 0 "C30" H 10550 5500 50  0000 L CNN
 F 1 "4.7u" H 10550 5300 50  0000 L CNN
-F 2 "Capacitors_SMD:C_0603_HandSoldering" H 10563 5250 50  0001 C CNN
+F 2 "Footprints_LJ:Cap_0603_HandSoldering_1" H 10563 5250 50  0001 C CNN
 F 3 "" H 10525 5400 50  0001 C CNN
 	1    10525 5400
@@
 F 0 "C31" H 10750 5500 50  0000 L CNN
 F 1 "0.47u" H 10750 5300 50  0000 L CNN
-F 2 "Capacitors_SMD:C_0603_HandSoldering" H 10763 5250 50  0001 C CNN
+F 2 "Footprints_LJ:Cap_0603_HandSoldering_1" H 10763 5250 50  0001 C CNN
 F 3 "" H 10725 5400 50  0001 C CNN
 	1    10725 5400
@@
 F 0 "C32" H 10950 5500 50  0000 L CNN
 F 1 "0.47u" H 10950 5300 50  0000 L CNN
-F 2 "Capacitors_SMD:C_0603_HandSoldering" H 10963 5250 50  0001 C CNN
+F 2 "Footprints_LJ:Cap_0603_HandSoldering_1" H 10963 5250 50  0001 C CNN
 F 3 "" H 10925 5400 50  0001 C CNN
 	1    10925 5400
@@
 F 0 "C33" H 10550 6225 50  0000 L CNN
 F 1 "4.7u" H 10550 6025 50  0000 L CNN
-F 2 "Capacitors_SMD:C_0603_HandSoldering" H 10563 5975 50  0001 C CNN
+F 2 "Footprints_LJ:Cap_0603_HandSoldering_1" H 10563 5975 50  0001 C CNN
 F 3 "" H 10525 6125 50  0001 C CNN
 	1    10525 6125
@@
 F 0 "C34" H 10750 6225 50  0000 L CNN
 F 1 "0.47u" H 10750 6025 50  0000 L CNN
-F 2 "Capacitors_SMD:C_0603_HandSoldering" H 10763 5975 50  0001 C CNN
+F 2 "Footprints_LJ:Cap_0603_HandSoldering_1" H 10763 5975 50  0001 C CNN
 F 3 "" H 10725 6125 50  0001 C CNN
 	1    10725 6125
@@
 F 0 "C35" H 10950 6225 50  0000 L CNN
 F 1 "0.47u" H 10950 6025 50  0000 L CNN
-F 2 "Capacitors_SMD:C_0603_HandSoldering" H 10963 5975 50  0001 C CNN
+F 2 "Footprints_LJ:Cap_0603_HandSoldering_1" H 10963 5975 50  0001 C CNN
 F 3 "" H 10925 6125 50  0001 C CNN
 	1    10925 6125
@@
 F 0 "C12" H 9325 1225 50  0000 L CNN
 F 1 "4.7u" H 9325 1025 50  0000 L CNN
-F 2 "Capacitors_SMD:C_0603_HandSoldering" H 9338 975 50  0001 C CNN
+F 2 "Footprints_LJ:Cap_0603_HandSoldering_1" H 9338 975 50  0001 C CNN
 F 3 "" H 9300 1125 50  0001 C CNN
 	1    9300 1125
@@
 F 0 "C13" H 9525 1225 50  0000 L CNN
 F 1 "4.7u" H 9525 1025 50  0000 L CNN
-F 2 "Capacitors_SMD:C_0603_HandSoldering" H 9538 975 50  0001 C CNN
+F 2 "Footprints_LJ:Cap_0603_HandSoldering_1" H 9538 975 50  0001 C CNN
 F 3 "" H 9500 1125 50  0001 C CNN
 	1    9500 1125
@@
 F 0 "C14" H 9725 1225 50  0000 L CNN
 F 1 "4.7u" H 9725 1025 50  0000 L CNN
-F 2 "Capacitors_SMD:C_0603_HandSoldering" H 9738 975 50  0001 C CNN
+F 2 "Footprints_LJ:Cap_0603_HandSoldering_1" H 9738 975 50  0001 C CNN
 F 3 "" H 9700 1125 50  0001 C CNN
 	1    9700 1125
@@
 F 0 "C15" H 9925 1225 50  0000 L CNN
 F 1 "4.7u" H 9925 1025 50  0000 L CNN
-F 2 "Capacitors_SMD:C_0603_HandSoldering" H 9938 975 50  0001 C CNN
+F 2 "Footprints_LJ:Cap_0603_HandSoldering_1" H 9938 975 50  0001 C CNN
 F 3 "" H 9900 1125 50  0001 C CNN
 	1    9900 1125
@@
 F 0 "C16" H 10125 1225 50  0000 L CNN
 F 1 "4.7u" H 10125 1025 50  0000 L CNN
-F 2 "Capacitors_SMD:C_0603_HandSoldering" H 10138 975 50  0001 C CNN
+F 2 "Footprints_LJ:Cap_0603_HandSoldering_1" H 10138 975 50  0001 C CNN
 F 3 "" H 10100 1125 50  0001 C CNN
 	1    10100 1125
@@
 F 0 "C17" H 10325 1225 50  0000 L CNN
 F 1 "4.7u" H 10325 1025 50  0000 L CNN
-F 2 "Capacitors_SMD:C_0603_HandSoldering" H 10338 975 50  0001 C CNN
+F 2 "Footprints_LJ:Cap_0603_HandSoldering_1" H 10338 975 50  0001 C CNN
 F 3 "" H 10300 1125 50  0001 C CNN
 	1    10300 1125
@@
 F 0 "C18" H 10525 1225 50  0000 L CNN
 F 1 "0.47u" H 10525 1025 50  0000 L CNN
-F 2 "Capacitors_SMD:C_0603_HandSoldering" H 10538 975 50  0001 C CNN
+F 2 "Footprints_LJ:Cap_0603_HandSoldering_1" H 10538 975 50  0001 C CNN
 F 3 "" H 10500 1125 50  0001 C CNN
 	1    10500 1125
@@
 F 0 "C20" H 9125 1925 50  0000 L CNN
 F 1 "4.7u" H 9125 1725 50  0000 L CNN
-F 2 "Capacitors_SMD:C_0603_HandSoldering" H 9138 1675 50  0001 C CNN
+F 2 "Footprints_LJ:Cap_0603_HandSoldering_1" H 9138 1675 50  0001 C CNN
 F 3 "" H 9100 1825 50  0001 C CNN
 	1    9100 1825
@@
 F 0 "C21" H 9325 1925 50  0000 L CNN
 F 1 "4.7u" H 9325 1725 50  0000 L CNN
-F 2 "Capacitors_SMD:C_0603_HandSoldering" H 9338 1675 50  0001 C CNN
+F 2 "Footprints_LJ:Cap_0603_HandSoldering_1" H 9338 1675 50  0001 C CNN
 F 3 "" H 9300 1825 50  0001 C CNN
 	1    9300 1825
@@
 F 0 "C22" H 9525 1925 50  0000 L CNN
 F 1 "0.47u" H 9525 1725 50  0000 L CNN
-F 2 "Capacitors_SMD:C_0603_HandSoldering" H 9538 1675 50  0001 C CNN
+F 2 "Footprints_LJ:Cap_0603_HandSoldering_1" H 9538 1675 50  0001 C CNN
 F 3 "" H 9500 1825 50  0001 C CNN
 	1    9500 1825
@@
 F 0 "C26" H 10125 5500 50  0000 L CNN
 F 1 "0.47u" H 10125 5300 50  0000 L CNN
-F 2 "Capacitors_SMD:C_0603_HandSoldering" H 10138 5250 50  0001 C CNN
+F 2 "Footprints_LJ:Cap_0603_HandSoldering_1" H 10138 5250 50  0001 C CNN
 F 3 "" H 10100 5400 50  0001 C CNN
 	1    10100 5400
@@
 F 0 "C8" H 4875 2475 50  0000 L CNN
 F 1 "1u" H 4875 2275 50  0000 L CNN
-F 2 "Capacitors_SMD:C_0603_HandSoldering" H 4888 2225 50  0001 C CNN
+F 2 "Footprints_LJ:Cap_0603_HandSoldering_1" H 4888 2225 50  0001 C CNN
 F 3 "" H 4850 2375 50  0001 C CNN
 	1    4850 2375
@@
 F 0 "C_TP_2" H 3200 6350 50  0000 L CNN
 F 1 "1u" H 3200 6150 50  0000 L CNN
-F 2 "Capacitors_SMD:C_0603_HandSoldering" H 3213 6100 50  0001 C CNN
+F 2 "Footprints_LJ:Cap_0603_HandSoldering_1" H 3213 6100 50  0001 C CNN
 F 3 "" H 3175 6250 50  0001 C CNN
 	1    3175 6250
@@
 F 0 "C_TP_1" H 2875 6350 50  0000 L CNN
 F 1 "1u" H 2875 6150 50  0000 L CNN
-F 2 "Capacitors_SMD:C_0603_HandSoldering" H 2888 6100 50  0001 C CNN
+F 2 "Footprints_LJ:Cap_0603_HandSoldering_1" H 2888 6100 50  0001 C CNN
 F 3 "" H 2850 6250 50  0001 C CNN
 	1    2850 6250
@@
 F 0 "C_I2C_2" H 4600 1350 50  0000 L CNN
 F 1 "1u" H 4600 1150 50  0000 L CNN
-F 2 "Capacitors_SMD:C_0603_HandSoldering" H 4613 1100 50  0001 C CNN
+F 2 "Footprints_LJ:Cap_0603_HandSoldering_1" H 4613 1100 50  0001 C CNN
 F 3 "" H 4575 1250 50  0001 C CNN
 	1    4575 1250
@@
 F 0 "C_I2C_1" H 4100 1350 50  0000 L CNN
 F 1 "1u" H 4100 1150 50  0000 L CNN
-F 2 "Capacitors_SMD:C_0603_HandSoldering" H 4113 1100 50  0001 C CNN
+F 2 "Footprints_LJ:Cap_0603_HandSoldering_1" H 4113 1100 50  0001 C CNN
 F 3 "" H 4075 1250 50  0001 C CNN
 	1    4075 1250
@@
 F 0 "C_JTAG_2" H 8325 5975 50  0000 L CNN
 F 1 "1u" H 8325 5775 50  0000 L CNN
-F 2 "Capacitors_SMD:C_0603_HandSoldering" H 8338 5725 50  0001 C CNN
+F 2 "Footprints_LJ:Cap_0603_HandSoldering_1" H 8338 5725 50  0001 C CNN
 F 3 "" H 8300 5875 50  0001 C CNN
 	1    8300 5875
@@
 F 0 "C_JTAG_1" H 7900 5975 50  0000 L CNN
 F 1 "1u" H 7900 5775 50  0000 L CNN
-F 2 "Capacitors_SMD:C_0603_HandSoldering" H 7913 5725 50  0001 C CNN
+F 2 "Footprints_LJ:Cap_0603_HandSoldering_1" H 7913 5725 50  0001 C CNN
 F 3 "" H 7875 5875 50  0001 C CNN
 	1    7875 5875
@@
 F 0 "C_RS2232_2" H 4900 3650 50  0000 L CNN
 F 1 "1u" H 4900 3450 50  0000 L CNN
-F 2 "Capacitors_SMD:C_0603_HandSoldering" H 4913 3400 50  0001 C CNN
+F 2 "Footprints_LJ:Cap_0603_HandSoldering_1" H 4913 3400 50  0001 C CNN
 F 3 "" H 4875 3550 50  0001 C CNN
 	1    4875 3550
@@
 F 0 "C_RS2232_1" H 4350 3650 50  0000 L CNN
 F 1 "1u" H 4350 3450 50  0000 L CNN
-F 2 "Capacitors_SMD:C_0603_HandSoldering" H 4363 3400 50  0001 C CNN
+F 2 "Footprints_LJ:Cap_0603_HandSoldering_1" H 4363 3400 50  0001 C CNN
 F 3 "" H 4325 3550 50  0001 C CNN
 	1    4325 3550
