File: kicad/FrequnecyCounter.kicad_pcb (KiCad board)
At the start: 2 copper layers, 150 x 90 mm, 160 parts, among them J1 USB_B, J2 CONN_COAXIAL, J3 CONN_COAXIAL, J4 CONN_COAXIAL, SW1 SW_Push, T1 WBC16-1T, T2 WBC16-1T, U1 TPS650250, U10 MC12093, U11 LTC6957-3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

Commit message: layout [in progress]
Parts:
- removed the REF** at (90.5, 130.8)
- removed the REF** at (98.1, 122.7)
- removed the REF** at (93.8, 135.0)
- removed the REF** at (84.1, 124.1)
- removed the REF** at (89.4, 128.0)
- removed the REF** at (92.1, 126.2)
- removed the REF** at (79.3, 112.8)
- removed the REF** at (76.6, 112.8)
- removed the REF** at (78.3, 122.6)
- added D11: LED, Footprints_LJ:Mini_TopLed_SMD, F.Cu at (117.5, 60.1)
- added R39: 680R, Resistors_SMD:R_0603_HandSoldering, F.Cu at (117.5, 65.2)
- added X1: Stiftleiste_2x10Pm_R2.54, Footprints_LJ:Stiftleiste_2x10Pm_R2.54, F.Cu at (170.1, 64.6)
- C15, C30, C7, R13: moved to B.Cu
- R7: value 33k -> 22k
- moved SW1 36.1 mm to (82.7, 93.6)
- moved R3 35.2 mm to (80.0, 106.9), turned to 180 degrees
- moved R8 16.6 mm to (112.8, 116.0), turned to 90 degrees
- moved C7 13.3 mm to (96.6, 130.1), turned to 0 degrees
- moved U3 11.6 mm to (116.3, 116.0), turned to 90 degrees
- moved C38 10.8 mm to (86.7, 76.3), turned to 0 degrees
- moved R1 10.3 mm to (85.3, 123.0), turned to 270 degrees
- moved C10 9.92 mm to (122.6, 128.4), turned to 270 degrees
- moved R9 9.83 mm to (120.9, 116.3), turned to 90 degrees
- moved C39 7.79 mm to (86.7, 78.0), turned to 0 degrees
- moved R10 7.52 mm to (107.7, 136.4), turned to 0 degrees
- moved C19 7.37 mm to (119.4, 116.4), turned to 90 degrees
- moved R4 6.69 mm to (82.2, 123.0), turned to 90 degrees
- moved C5 6.57 mm to (103.8, 117.6), turned to 270 degrees
- moved C1 6.30 mm to (82.6, 117.6), turned to 270 degrees
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Connections:
- net +3.6V renamed +3V6
- C11 pad 1: +2V5 -> +3V3_FPGA
- C12 pad 1: +2V5 -> +3V3_FPGA
- C13 pad 1: +2V5 -> +3V3_FPGA
- C14 pad 1: +2V5 -> +3V3_FPGA
- C15 pad 1: +2V5 -> +3V3_FPGA
- C16 pad 1: +2V5 -> +3V3_FPGA
- C17 pad 1: +2V5 -> +3V3_FPGA
- C18 pad 1: +2V5 -> +3V3_FPGA
- C19 pad 1: +3V3 -> +3V3_FPGA
- C24 pad 1: +3V3 -> +3V3_FPGA
- C25 pad 1: +3V3 -> +3V3_FPGA
- C26 pad 1: +3V3 -> +3V3_FPGA
- C27 pad 1: +3V3 -> +3V3_FPGA
- C28 pad 1: +3V3 -> +3V3_FPGA
- C29 pad 1: +3V3 -> +3V3_FPGA
- C30 pad 1: +3V3 -> +3V3_FPGA
- C31 pad 1: +3V3 -> +3V3_FPGA
- C32 pad 1: +3V3 -> +3V3_FPGA
- C33 pad 1: +3V3 -> +3V3_FPGA
- C34 pad 1: +3V3 -> +3V3_FPGA
- C35 pad 1: +3V3 -> +3V3_FPGA
- C5 pad 1: +2V5 -> +3V3_FPGA
- C6 pad 1: +2V5 -> +3V3_FPGA
- G1 pad 8: /FPGA/Ref_Clk -> Int_Ref_Clk
- L3 pad 2: +2V5 -> +3V3_FPGA
- R11 pad 1: +3V3 -> +3V3_FPGA
- R12 pad 1: +3V3 -> +3V3_FPGA
- R13 pad 1: +3V3 -> +3V3_FPGA
- R5 pad 1: +2V5 -> +3V3_FPGA
- R8 pad 1: +3V3 -> +3V3_FPGA
- R9 pad 1: +3V3 -> +3V3_FPGA
- U1 pad 1: +2V5 -> +3V3_FPGA
- U3 pad 3: +3V3 -> +3V3_FPGA
- U6 pad 10: +3V3 -> Net-(U6-Pad10)
- xc6slx9_1 pad 10: /Signal_Input/CHA_FILTA -> Net-(xc6slx9_1-Pad10)
- xc6slx9_1 pad 103: +3V3 -> +3V3_FPGA
- xc6slx9_1 pad 11: Net-(xc6slx9_1-Pad11) -> TP10
- xc6slx9_1 pad 12: /Signal_Input/CHA_FILTB -> TP9
- xc6slx9_1 pad 122: +3V3 -> +3V3_FPGA
- xc6slx9_1 pad 123: Net-(xc6slx9_1-Pad123) -> Int_Ref_Clk
- xc6slx9_1 pad 124: /FPGA/Ref_Clk -> /FPGA/Clk_A
- xc6slx9_1 pad 125: +3V3 -> +3V3_FPGA
- xc6slx9_1 pad 126: Net-(xc6slx9_1-Pad126) -> /Signal_Input/CHA_FILTA
- xc6slx9_1 pad 127: /FPGA/Clk_A -> /FPGA/Ext_Ref_Clk
- xc6slx9_1 pad 129: +2V5 -> +3V3_FPGA
- xc6slx9_1 pad 131: Net-(xc6slx9_1-Pad131) -> /Signal_Input/CHA_FILTB
- xc6slx9_1 pad 132: /FPGA/Ext_Ref_Clk -> /FPGA/Clk_B
- xc6slx9_1 pad 133: Net-(xc6slx9_1-Pad133) -> /Signal_Input/CHB_FILTB
- xc6slx9_1 pad 134: /FPGA/Clk_B -> /Signal_Input/CHB_FILTA
- xc6slx9_1 pad 135: +3V3 -> +3V3_FPGA
- xc6slx9_1 pad 14: Net-(xc6slx9_1-Pad14) -> TP8
- xc6slx9_1 pad 15: Net-(xc6slx9_1-Pad15) -> TP7
- xc6slx9_1 pad 16: Net-(xc6slx9_1-Pad16) -> TP6
- xc6slx9_1 pad 17: Net-(xc6slx9_1-Pad17) -> TP5
- xc6slx9_1 pad 18: +3V3 -> +3V3_FPGA
- xc6slx9_1 pad 20: +2V5 -> +3V3_FPGA
- xc6slx9_1 pad 21: Net-(xc6slx9_1-Pad21) -> TP4
- xc6slx9_1 pad 22: Net-(xc6slx9_1-Pad22) -> TP3
- xc6slx9_1 pad 23: Net-(xc6slx9_1-Pad23) -> TP2
- xc6slx9_1 pad 24: Net-(xc6slx9_1-Pad24) -> TP1
- xc6slx9_1 pad 31: +3V3 -> +3V3_FPGA
- xc6slx9_1 pad 33: LED7 -> Net-(xc6slx9_1-Pad33)
- xc6slx9_1 pad 34: LED6 -> Net-(xc6slx9_1-Pad34)
- xc6slx9_1 pad 35: LED5 -> Net-(xc6slx9_1-Pad35)
- xc6slx9_1 pad 36: +2V5 -> +3V3_FPGA
- xc6slx9_1 pad 4: +3V3 -> +3V3_FPGA
- xc6slx9_1 pad 42: +3V3 -> +3V3_FPGA
- xc6slx9_1 pad 48: Net-(xc6slx9_1-Pad48) -> LED7
- xc6slx9_1 pad 50: Net-(xc6slx9_1-Pad50) -> LED6
- xc6slx9_1 pad 51: Net-(xc6slx9_1-Pad51) -> LED5
- xc6slx9_1 pad 53: +2V5 -> +3V3_FPGA
- xc6slx9_1 pad 6: /Signal_Input/CHB_FILTB -> Net-(xc6slx9_1-Pad6)
- xc6slx9_1 pad 60: +3V3 -> +3V3_FPGA
- xc6slx9_1 pad 63: +3V3 -> +3V3_FPGA
- xc6slx9_1 pad 69: +3V3 -> +3V3_FPGA
- xc6slx9_1 pad 76: +3V3 -> +3V3_FPGA
- xc6slx9_1 pad 8: /Signal_Input/CHB_FILTA -> Net-(xc6slx9_1-Pad8)
- xc6slx9_1 pad 86: +3V3 -> +3V3_FPGA
- xc6slx9_1 pad 90: +2V5 -> +3V3_FPGA
Routing:
- net +3V3: track 621.3 -> 288.6 mm, vias 28 -> 9
- net +3V3_FPGA: track 0.00 -> 306.2 mm, vias 0 -> 17
- net +2V5: track 160.8 -> 0.00 mm, vias 6 -> 0
- net /FPGA/Ref_Clk: track 37.0 -> 0.00 mm
- net +1.2V: track 207.4 -> 172.1 mm, vias 4 -> 5
- net Int_Ref_Clk: track 0.00 -> 31.4 mm
- net /Power_Supply/~RESET: track 98.3 -> 67.1 mm, vias 5 -> 3
- net TP10: track 0.00 -> 29.5 mm
- net TP8: track 0.00 -> 27.8 mm
- net TP6: track 0.00 -> 26.3 mm
- net TP9: track 0.00 -> 25.8 mm
- net TP4: track 0.00 -> 24.2 mm
- net TP7: track 0.00 -> 24.2 mm
- net TP2: track 0.00 -> 22.8 mm
- net TP5: track 0.00 -> 22.7 mm
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Other:
- copper layers 2 -> 4

Commit message: Layout changes [In progress]
Parts:
- removed D10, D3, D4, D9: LED, Footprints_LJ:Mini_TopLed_SMD
- removed R17, R22, R23: 680R, Resistors_SMD:R_0603_HandSoldering
- removed the REF** at (183.1, 102.8)
- added C8: 1u, Capacitors_SMD:C_0603_HandSoldering, F.Cu at (131.9, 135.2)
- C21: moved to B.Cu
- R16: value 680R -> 1k
- moved R16 67.8 mm to (131.8, 132.8), turned to 0 degrees
- moved C7 42.7 mm to (57.8, 112.4)
- moved C18 23.7 mm to (140.5, 108.2)
- moved C13 22.8 mm to (169.0, 85.4), turned to 45 degrees
- moved C20 21.7 mm to (150.0, 96.0), turned to 90 degrees
- moved C11 19.8 mm to (157.3, 73.7), turned to 45 degrees
- moved C16 18.9 mm to (137.7, 78.6), turned to 135 degrees
- moved C19 18.7 mm to (138.1, 118.5)
- moved R8 18.7 mm to (131.4, 118.1)
- moved R9 18.7 mm to (139.5, 118.4)
- moved U3 18.7 mm to (134.9, 118.1)
- moved C21 17.2 mm to (153.8, 92.0), turned to 180 degrees
- moved C14 15.6 mm to (138.7, 77.6), turned to 135 degrees
- moved C17 14.6 mm to (157.6, 109.7), turned to 315 degrees
- moved C12 12.8 mm to (167.1, 100.2), turned to 315 degrees
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Connections:
- C19 pad 1: +3V3_FPGA -> +3V3
- G1 pad 1: Net-(G1-Pad1) -> Net-(C8-Pad1)
- R16 pad 1: LED0 -> Net-(R16-Pad1)
- R16 pad 2: Net-(D3-Pad2) -> Net-(C8-Pad1)
- R18 pad 1: LED2 -> LED0
- R19 pad 1: LED3 -> LED1
- R20 pad 1: LED4 -> LED2
- R21 pad 1: LED5 -> LED3
- R8 pad 1: +3V3_FPGA -> +3V3
- R9 pad 1: +3V3_FPGA -> +3V3
- U1 pad 33: GND -> (no net)
- U3 pad 1: Net-(G1-Pad1) -> Net-(R16-Pad1)
- U3 pad 3: +3V3_FPGA -> +3V3
- U6 pad 10: Net-(U6-Pad10) -> +3V3
- U6 pad 26: Net-(U6-Pad26) -> +3V3
- xc6slx9_1 pad 48: LED7 -> Net-(xc6slx9_1-Pad48)
- xc6slx9_1 pad 50: LED6 -> Net-(xc6slx9_1-Pad50)
- xc6slx9_1 pad 51: LED5 -> Net-(xc6slx9_1-Pad51)
- xc6slx9_1 pad 55: LED4 -> Net-(xc6slx9_1-Pad55)
- xc6slx9_1 pad 60: +3V3_FPGA -> GND
- xc6slx9_1 pad 80: /FPGA/RXD -> Net-(xc6slx9_1-Pad80)
- xc6slx9_1 pad 82: /USB_JTAG/RXD -> Net-(xc6slx9_1-Pad82)
- xc6slx9_1 pad 84: Net-(xc6slx9_1-Pad84) -> /FPGA/RXD
- xc6slx9_1 pad 85: Net-(xc6slx9_1-Pad85) -> /USB_JTAG/RXD
Routing:
- net (no net): track 0.00 -> 769.3 mm
- net +3V3: track 288.6 -> 81.1 mm, vias 9 -> 14
- net +3V3_FPGA: track 306.2 -> 137.1 mm, vias 17 -> 22
- net +1.2V: track 172.1 -> 45.9 mm, vias 5 -> 9
- net Net-(G1-Pad1): track 33.3 -> 0.00 mm, vias 2 -> 0
- net SDA_DAC: track 37.6 -> 68.6 mm
- net SCL_DAC: track 40.4 -> 68.0 mm
- net LED5: track 19.7 -> 0.00 mm
- net LED4: track 19.6 -> 0.00 mm
- net LED7: track 18.3 -> 0.00 mm
- net LED6: track 18.1 -> 0.00 mm
- net Net-(R16-Pad1): track 0.00 -> 14.7 mm, vias 0 -> 2
- net +5V: track 131.5 -> 120.9 mm
- net +3V6: track 45.9 -> 53.7 mm
- net Net-(C8-Pad1): track 0.00 -> 7.67 mm
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- added copper zone on In2.Cu, net GND

Commit message: Layout changes [in progress]
Parts:
- removed C52, C53: 100n, Capacitors_SMD:C_0603_HandSoldering
- removed D5, D6, D7, D8: LED, Footprints_LJ:Mini_TopLed_SMD
- removed R18, R19, R20, R21: 680R, Resistors_SMD:R_0603_HandSoldering
- removed R37: 47R, Resistors_SMD:R_0603_HandSoldering
- removed R38: 100R, Resistors_SMD:R_0603_HandSoldering
- removed the REF** at (205.0, 87.7)
- removed the REF** at (204.2, 87.7)
- removed the REF** at (203.4, 87.7)
- removed the REF** at (205.0, 88.5)
- removed the REF** at (204.2, 88.5)
- removed the REF** at (203.4, 88.5)
- removed T2: WBC16-1T, Footprints_LJ:wbc-16-1T
- removed V2: HSMS-281C-TR1G, TO_SOT_Packages_SMD:SOT-323_SC-70_Handsoldering
- added D3: BAV99, TO_SOT_Packages_SMD:SOT-23, F.Cu at (169.4, 126.9)
- added D4: BAV99, TO_SOT_Packages_SMD:SOT-23, F.Cu at (196.8, 120.1)
- added R17: 680R, Resistors_SMD:R_0603_HandSoldering, F.Cu at (169.4, 112.5)
- added R22: 680R, Resistors_SMD:R_0603_HandSoldering, F.Cu at (169.4, 110.2)
- added R23: 1k, Resistors_SMD:R_0603_HandSoldering, F.Cu at (190.8, 128.9)
- added U12: TLV3501, SMD_Packages:SOIC-8-N, F.Cu at (190.4, 121.0)
- added U13: ADR5040, TO_SOT_Packages_SMD:SOT-323_SC-70_Handsoldering, F.Cu at (190.6, 126.1)
- C11, C12, C13, C14, C15, C16, C17, C18, C24, C25, C26, C27, C28, C29, C30, C31, C32, C33, C34, C35, C36, C7, R13, R24: moved to F.Cu
- C51: value 100n -> 100p
- R35: value 100R -> 100k
- R36: value 560R -> 1k
- U11: value LTC6957-3 -> tx176; footprint Housings_DFN_QFN:DFN-12-1EP_3x3mm_Pitch0.45mm -> Footprints_LJ:tx176
- U7: footprint Crystal_HC49-U_Vertical -> Crystals:Crystal_HC49-U_Vertical
- moved G1 79.2 mm to (170.4, 62.8), turned to 180 degrees
- moved X1 73.3 mm to (142.6, 132.5), turned to 180 degrees
- moved C23 70.5 mm to (175.0, 71.4)
- moved C8 70.4 mm to (169.4, 75.6), turned to 270 degrees
- moved R16 67.4 mm to (167.6, 75.8), turned to 90 degrees
- moved R8 52.7 mm to (170.1, 82.4), turned to 270 degrees
- moved R4 51.1 mm to (127.6, 122.8)
- moved C1 51.1 mm to (129.2, 116.5)
- moved C2 51.1 mm to (126.4, 116.5)
- moved R1 51.1 mm to (127.6, 120.6)
- moved C7 50.4 mm to (108.0, 116.9), turned to 90 degrees
- moved U3 47.8 mm to (166.6, 82.4), turned to 270 degrees
- moved U11 45.6 mm to (165.3, 64.4), turned to 180 degrees
- moved C19 44.4 mm to (163.4, 82.0), turned to 270 degrees
- moved R9 42.6 mm to (162.0, 82.1), turned to 270 degrees
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Connections:
- net Net-(xc6slx9_1-Pad32) renamed /FPGA/EN_CHB_FILTB
- net Net-(xc6slx9_1-Pad34) renamed /FPGA/EN_CHB_FILTA
- C50 pad 1: Net-(C50-Pad1) -> +3V3
- C50 pad 2: /Signal_Input/CHB+ -> GND
- C51 pad 1: Net-(C51-Pad1) -> /FPGA/Clk_A
- C51 pad 2: /Signal_Input/CH_B -> Net-(C51-Pad2)
- R35 pad 1: /Signal_Input/CHB+ -> Net-(R23-Pad1)
- R35 pad 2: /Signal_Input/T2+ -> Net-(R35-Pad2)
- R36 pad 1: /Signal_Input/CHB+ -> Net-(R35-Pad2)
- R36 pad 2: Net-(R36-Pad2) -> GND
- U1 pad 1: +3V3_FPGA -> +1.2V
- U1 pad 22: Net-(R2-Pad2) -> Net-(R5-Pad2)
- U1 pad 25: +3V6 -> +3V3_FPGA
- U1 pad 27: Net-(L2-Pad1) -> Net-(L3-Pad1)
- U1 pad 3: Net-(L3-Pad1) -> Net-(L1-Pad1)
- U1 pad 32: Net-(R5-Pad2) -> Net-(R1-Pad2)
- U1 pad 6: Net-(L1-Pad1) -> Net-(L2-Pad1)
- U1 pad 8: +1.2V -> +3V6
- U1 pad 9: Net-(R1-Pad2) -> Net-(R2-Pad2)
- U10 pad 4: /FPGA/Clk_A -> Net-(C51-Pad2)
- U11 pad 10: /FPGA/Clk_B -> Net-(C8-Pad1)
- U11 pad 4: Net-(C52-Pad1) -> GND
- U11 pad 5: GND -> Int_Ref_Clk
- U11 pad 9: Net-(U11-Pad9) -> +3V3
- xc6slx9_1 pad 10: Net-(xc6slx9_1-Pad10) -> /Signal_Input/CHA_FILTA
- xc6slx9_1 pad 11: TP10 -> Net-(xc6slx9_1-Pad11)
- xc6slx9_1 pad 12: TP9 -> Net-(xc6slx9_1-Pad12)
- xc6slx9_1 pad 120: Net-(xc6slx9_1-Pad120) -> TP10
- xc6slx9_1 pad 121: Net-(xc6slx9_1-Pad121) -> TP9
- xc6slx9_1 pad 123: Int_Ref_Clk -> TP8
- xc6slx9_1 pad 124: /FPGA/Clk_A -> TP7
- xc6slx9_1 pad 126: /Signal_Input/CHA_FILTA -> TP6
- xc6slx9_1 pad 127: /FPGA/Ext_Ref_Clk -> TP5
- xc6slx9_1 pad 131: /Signal_Input/CHA_FILTB -> TP4
- xc6slx9_1 pad 132: /FPGA/Clk_B -> TP3
- xc6slx9_1 pad 133: /Signal_Input/CHB_FILTB -> TP2
- xc6slx9_1 pad 134: /Signal_Input/CHB_FILTA -> TP1
- xc6slx9_1 pad 14: TP8 -> /FPGA/Clk_A
- xc6slx9_1 pad 15: TP7 -> Net-(xc6slx9_1-Pad15)
- xc6slx9_1 pad 16: TP6 -> /FPGA/Ext_Ref_Clk
- xc6slx9_1 pad 17: TP5 -> Net-(xc6slx9_1-Pad17)
- xc6slx9_1 pad 21: TP4 -> /FPGA/Clk_B
- xc6slx9_1 pad 22: TP3 -> Net-(xc6slx9_1-Pad22)
- xc6slx9_1 pad 23: TP2 -> SCL_DAC
- xc6slx9_1 pad 24: TP1 -> SDA_DAC
- xc6slx9_1 pad 46: Net-(xc6slx9_1-Pad46) -> LED3
- xc6slx9_1 pad 50: Net-(xc6slx9_1-Pad50) -> Int_Ref_Clk
- xc6slx9_1 pad 56: LED3 -> LED2
- xc6slx9_1 pad 57: LED2 -> Net-(xc6slx9_1-Pad57)
- xc6slx9_1 pad 58: LED1 -> Net-(xc6slx9_1-Pad58)
- xc6slx9_1 pad 59: LED0 -> LED1
- xc6slx9_1 pad 62: Net-(xc6slx9_1-Pad62) -> LED0
- xc6slx9_1 pad 8: Net-(xc6slx9_1-Pad8) -> /Signal_Input/CHA_FILTB
- xc6slx9_1 pad 84: /FPGA/RXD -> Net-(xc6slx9_1-Pad84)
- xc6slx9_1 pad 85: /USB_JTAG/RXD -> Net-(xc6slx9_1-Pad85)
- xc6slx9_1 pad 87: Net-(xc6slx9_1-Pad87) -> /FPGA/RXD
- xc6slx9_1 pad 88: Net-(xc6slx9_1-Pad88) -> /USB_JTAG/RXD
- xc6slx9_1 pad 93: SCL_DAC -> Net-(xc6slx9_1-Pad93)
- xc6slx9_1 pad 94: SDA_DAC -> Net-(xc6slx9_1-Pad94)
Routing:
- net /Signal_Input/CHB_FILTA: track 60.5 -> 0.00 mm, vias 2 -> 0
- net /Signal_Input/CHB_FILTB: track 53.6 -> 0.00 mm, vias 2 -> 0
- net LED0: track 23.3 -> 0.01 mm
- net LED1: track 21.7 -> 0.00 mm
- net WORK_LED: track 25.9 -> 4.32 mm, vias 0 -> 2
- net LED2: track 20.3 -> 0.00 mm
- net +3V6: track 53.7 -> 33.6 mm
- net /FPGA/Clk_A: track 39.7 -> 20.7 mm, vias 2 -> 0
- net LED3: track 19.0 -> 0.92 mm
- net /FPGA/TCK: track 70.1 -> 52.4 mm, vias 0 -> 2
- net DONE_LED: track 30.6 -> 12.9 mm
- net /FPGA/TDI: track 75.0 -> 57.5 mm, vias 0 -> 2
- net +3V3: track 81.1 -> 64.5 mm, vias 14 -> 18
- net Net-(R10-Pad2): track 19.5 -> 3.35 mm
- net +5V: track 120.9 -> 136.6 mm, vias 6 -> 5
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
Commit message: Reworked schematic and layout [to review]
Parts:
- moved X1 55.4 mm to (187.2, 99.8), turned to 90 degrees
- moved C23 27.6 mm to (147.3, 72.4)
- moved G1 27.6 mm to (142.8, 63.8)
- moved U11 27.6 mm to (137.6, 65.4)
- moved R17 27.3 mm to (144.1, 122.5), turned to 90 degrees
- moved R8 25.7 mm to (155.6, 61.2), turned to 0 degrees
- moved R22 25.1 mm to (147.6, 122.5), turned to 270 degrees
- moved C8 24.7 mm to (148.8, 62.0), turned to 0 degrees
- moved J3 23.8 mm to (146.7, 136.7)
- moved R16 22.1 mm to (148.9, 63.8), turned to 180 degrees
- moved C43 21.8 mm to (168.6, 89.7)
- moved R30 21.7 mm to (167.5, 74.6)
- moved R31 21.7 mm to (168.7, 84.4)
- moved R33 21.7 mm to (172.5, 74.6)
- moved V1 21.7 mm to (170.0, 80.4)
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Connections:
- net /FPGA/EN_CHB_FILTA renamed Net-(xc6slx9_1-Pad34)
- net /FPGA/EN_CHB_FILTB renamed Net-(xc6slx9_1-Pad32)
- net LED0 renamed Net-(xc6slx9_1-Pad62)
- net LED1 renamed Net-(xc6slx9_1-Pad59)
- net LED3 renamed Net-(xc6slx9_1-Pad46)
- U1 pad 33: (no net) -> GND
- U9 pad 1: /Signal_Input/CHA_FILTA -> /FPGA/EN_EXTREF_FILTA
- U9 pad 6: /Signal_Input/CHA_FILTB -> /FPGA/EN_EXTREF_FILTB
- X1 pad 1: SCL_DAC -> TP1
- X1 pad 10: TP8 -> TP10
- X1 pad 11: TP9 -> SCL_DAC
- X1 pad 12: TP10 -> SDA_DAC
- X1 pad 2: SDA_DAC -> TP2
- X1 pad 3: TP1 -> TP3
- X1 pad 4: TP2 -> TP4
- X1 pad 5: TP3 -> TP5
- X1 pad 6: TP4 -> TP6
- X1 pad 7: TP5 -> TP7
- X1 pad 8: TP6 -> TP8
- X1 pad 9: TP7 -> TP9
- xc6slx9_1 pad 10: /Signal_Input/CHA_FILTA -> Net-(xc6slx9_1-Pad10)
- xc6slx9_1 pad 120: TP10 -> Net-(xc6slx9_1-Pad120)
- xc6slx9_1 pad 121: TP9 -> Net-(xc6slx9_1-Pad121)
- xc6slx9_1 pad 123: TP8 -> Net-(xc6slx9_1-Pad123)
- xc6slx9_1 pad 124: TP7 -> Net-(xc6slx9_1-Pad124)
- xc6slx9_1 pad 126: TP6 -> Net-(xc6slx9_1-Pad126)
- xc6slx9_1 pad 127: TP5 -> Net-(xc6slx9_1-Pad127)
- xc6slx9_1 pad 131: TP4 -> Net-(xc6slx9_1-Pad131)
- xc6slx9_1 pad 132: TP3 -> Net-(xc6slx9_1-Pad132)
- xc6slx9_1 pad 133: TP2 -> Net-(xc6slx9_1-Pad133)
- xc6slx9_1 pad 134: TP1 -> /FPGA/Clk_A
- xc6slx9_1 pad 137: Net-(xc6slx9_1-Pad137) -> TP1
- xc6slx9_1 pad 138: Net-(xc6slx9_1-Pad138) -> TP2
- xc6slx9_1 pad 139: Net-(xc6slx9_1-Pad139) -> TP3
- xc6slx9_1 pad 14: /FPGA/Clk_A -> /FPGA/Clk_B
- xc6slx9_1 pad 140: Net-(xc6slx9_1-Pad140) -> TP4
- xc6slx9_1 pad 141: Net-(xc6slx9_1-Pad141) -> TP5
- xc6slx9_1 pad 15: Net-(xc6slx9_1-Pad15) -> SCL_DAC
- xc6slx9_1 pad 16: /FPGA/Ext_Ref_Clk -> SDA_DAC
- xc6slx9_1 pad 17: Net-(xc6slx9_1-Pad17) -> /FPGA/EN_EXTREF_FILTB
- xc6slx9_1 pad 21: /FPGA/Clk_B -> Net-(xc6slx9_1-Pad21)
- xc6slx9_1 pad 22: Net-(xc6slx9_1-Pad22) -> /FPGA/EN_EXTREF_FILTA
- xc6slx9_1 pad 23: SCL_DAC -> Net-(xc6slx9_1-Pad23)
- xc6slx9_1 pad 24: SDA_DAC -> /FPGA/Ext_Ref_Clk
- xc6slx9_1 pad 5: Net-(xc6slx9_1-Pad5) -> TP6
- xc6slx9_1 pad 50: Int_Ref_Clk -> Net-(xc6slx9_1-Pad50)
- xc6slx9_1 pad 56: LED2 -> Int_Ref_Clk
- xc6slx9_1 pad 6: Net-(xc6slx9_1-Pad6) -> TP7
- xc6slx9_1 pad 7: Net-(xc6slx9_1-Pad7) -> TP8
- xc6slx9_1 pad 8: /Signal_Input/CHA_FILTB -> TP9
- xc6slx9_1 pad 9: Net-(xc6slx9_1-Pad9) -> TP10
Routing:
- net /Signal_Input/CHA_FILTB: track 40.2 -> 0.00 mm, vias 2 -> 0
- net /Signal_Input/CHA_FILTA: track 35.5 -> 0.00 mm, vias 2 -> 0
- net WORK_LED: track 4.32 -> 34.6 mm
- net SCL_DAC: track 62.6 -> 91.5 mm
- net (no net): track 772.4 -> 744.6 mm
- net TP1: track 20.8 -> 47.9 mm, vias 0 -> 1
- net TP3: track 20.2 -> 46.2 mm, vias 0 -> 1
- net TP5: track 20.3 -> 45.3 mm
- net /FPGA/EN_EXTREF_FILTB: track 0.00 -> 21.6 mm
- net DONE_LED: track 12.9 -> 34.1 mm
- net TP2: track 23.6 -> 44.0 mm, vias 0 -> 1
- net TP4: track 22.9 -> 42.7 mm, vias 0 -> 1
- net SDA_DAC: track 66.4 -> 85.7 mm
- net +3V3_FPGA: track 132.8 -> 151.6 mm, vias 13 -> 16
- net /FPGA/Ext_Ref_Clk: track 38.0 -> 20.0 mm, vias 2 -> 0
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- added copper zone on In1.Cu, net +1.2V
- added copper zone on In1.Cu, net +3V3
- added copper zone on In1.Cu, net +3V3_FPGA
Other:
- board size 150 x 90 mm -> 130 x 90 mm
- net class Default: clearance 0.2 -> 0.16
- net class POWER: clearance 0.2 -> 0.16
- rule trace_clearance: 0.2 -> 0.16
