File: kicad/USB_JTAG.sch (KiCad schematic (older format))
At the start: 22 parts, among them J1 USB_B, Q1 BC846B, U4 NFM18PS, U5 WE-TVS-824011, U6 FT2232D, U7 6MHz_Crystal, U8 AT93C46DN-SH

Commit message: clean up in layout & add exports (assembly drawings)
Parts:
- C36, C37, C38, C39, C40, C41, C42: footprint Capacitors_SMD:C_0603_HandSoldering -> Footprints_LJ:Cap_0603_HandSoldering_1
Changed lines of the file:
@@
 F 0 "C40" V 4575 3975 50  0000 L CNN
 F 1 "27p" V 4500 3975 50  0000 L CNN
-F 2 "Capacitors_SMD:C_0603_HandSoldering" H 4738 3975 50  0001 C CNN
+F 2 "Footprints_LJ:Cap_0603_HandSoldering_1" H 4738 3975 50  0001 C CNN
 F 3 "" H 4700 4125 50  0001 C CNN
 	1    4700 4125
@@
 F 0 "C41" V 4825 4475 50  0000 L CNN
 F 1 "27p" V 4750 4475 50  0000 L CNN
-F 2 "Capacitors_SMD:C_0603_HandSoldering" H 4738 4175 50  0001 C CNN
+F 2 "Footprints_LJ:Cap_0603_HandSoldering_1" H 4738 4175 50  0001 C CNN
 F 3 "" H 4700 4325 50  0001 C CNN
 	1    4700 4325
@@
 F 0 "C37" V 5350 2575 50  0000 L CNN
 F 1 "33n" V 5275 2575 50  0000 L CNN
-F 2 "Capacitors_SMD:C_0603_HandSoldering" H 5263 2275 50  0001 C CNN
+F 2 "Footprints_LJ:Cap_0603_HandSoldering_1" H 5263 2275 50  0001 C CNN
 F 3 "" H 5225 2425 50  0001 C CNN
 	1    5225 2425
@@
 F 0 "C38" V 2200 3400 50  0000 L CNN
 F 1 "10u" V 2125 3400 50  0000 L CNN
-F 2 "Capacitors_SMD:C_0603_HandSoldering" H 2113 3100 50  0001 C CNN
+F 2 "Footprints_LJ:Cap_0603_HandSoldering_1" H 2113 3100 50  0001 C CNN
 F 3 "" H 2075 3250 50  0001 C CNN
 	1    2075 3250
@@
 F 0 "C36" V 5575 2025 50  0000 L CNN
 F 1 "33n" V 5500 2025 50  0000 L CNN
-F 2 "Capacitors_SMD:C_0603_HandSoldering" H 5488 1725 50  0001 C CNN
+F 2 "Footprints_LJ:Cap_0603_HandSoldering_1" H 5488 1725 50  0001 C CNN
 F 3 "" H 5450 1875 50  0001 C CNN
 	1    5450 1875
@@
 F 0 "C39" V 2525 3400 50  0000 L CNN
 F 1 "100n" V 2450 3400 50  0000 L CNN
-F 2 "Capacitors_SMD:C_0603_HandSoldering" H 2438 3100 50  0001 C CNN
+F 2 "Footprints_LJ:Cap_0603_HandSoldering_1" H 2438 3100 50  0001 C CNN
 F 3 "" H 2400 3250 50  0001 C CNN
 	1    2400 3250
@@
 F 0 "C42" H 2775 4875 50  0000 L CNN
 F 1 "100n" H 2775 4675 50  0000 L CNN
-F 2 "Capacitors_SMD:C_0603_HandSoldering" H 2788 4625 50  0001 C CNN
+F 2 "Footprints_LJ:Cap_0603_HandSoldering_1" H 2788 4625 50  0001 C CNN
 F 3 "" H 2750 4775 50  0001 C CNN
 	1    2750 4775
@@
 $EndComp
 $Comp
-L GND #PWR037
+L GND #PWR035
 U 1 1 5964E8AB
 P 2750 4925
-F 0 "#PWR037" H 2750 4675 50  0001 C CNN
+F 0 "#PWR035" H 2750 4675 50  0001 C CNN
 F 1 "GND" H 2750 4775 50  0000 C CNN
 F 2 "" H 2750 4925 50  0001 C CNN
@@
 $EndComp
 $Comp
-L +5V #PWR038
+L +5V #PWR036
 U 1 1 5968BBC0
 P 2075 1925
-F 0 "#PWR038" H 2075 1775 50  0001 C CNN
+F 0 "#PWR036" H 2075 1775 50  0001 C CNN
 F 1 "+5V" H 2075 2065 50  0000 C CNN
 F 2 "" H 2075 1925 50  0001 C CNN
@@
 $EndComp
 $Comp
-L +5V #PWR039
+L +5V #PWR037
 U 1 1 596B00B1
 P 6125 1700
-F 0 "#PWR039" H 6125 1550 50  0001 C CNN
+F 0 "#PWR037" H 6125 1550 50  0001 C CNN
 F 1 "+5V" H 6125 1840 50  0000 C CNN
 F 2 "" H 6125 1700 50  0001 C CNN
@@
 $EndComp
 $Comp
-L +5V #PWR040
+L +5V #PWR038
 U 1 1 596CAD7A
 P 4950 1675
-F 0 "#PWR040" H 4950 1525 50  0001 C CNN
+F 0 "#PWR038" H 4950 1525 50  0001 C CNN
 F 1 "+5V" H 4950 1815 50  0000 C CNN
 F 2 "" H 4950 1675 50  0001 C CNN
@@
 Connection ~ 4550 4325
 $Comp
-L GND #PWR041
+L GND #PWR039
 U 1 1 5973DDBE
 P 4550 4350
-F 0 "#PWR041" H 4550 4100 50  0001 C CNN
+F 0 "#PWR039" H 4550 4100 50  0001 C CNN
 F 1 "GND" H 4550 4200 50  0000 C CNN
 F 2 "" H 4550 4350 50  0001 C CNN
@@
 	7175 5025 7300 5025
 $Comp
-L +3.3V #PWR042
+L +3.3V #PWR040
 U 1 1 59C1476A
 P 7300 5025
-F 0 "#PWR042" H 7300 4875 50  0001 C CNN
+F 0 "#PWR040" H 7300 4875 50  0001 C CNN
 F 1 "+3.3V" H 7300 5165 50  0000 C CNN
 F 2 "" H 7300 5025 50  0001 C CNN
@@
 $EndComp
 $Comp
-L +5V #PWR043
+L +5V #PWR041
 U 1 1 59FCA280
 P 5050 3625
-F 0 "#PWR043" H 5050 3475 50  0001 C CNN
+F 0 "#PWR041" H 5050 3475 50  0001 C CNN
 F 1 "+5V" H 5050 3765 50  0000 C CNN
 F 2 "" H 5050 3625 50  0001 C CNN
@@
 	7175 3525 7300 3525
 $Comp
-L +3.3V #PWR044
+L +3.3V #PWR042
 U 1 1 59FCF531
 P 7300 3525
-F 0 "#PWR044" H 7300 3375 50  0001 C CNN
+F 0 "#PWR042" H 7300 3375 50  0001 C CNN
 F 1 "+3.3V" H 7300 3665 50  0000 C CNN
 F 2 "" H 7300 3525 50  0001 C CNN
@@
 	7750 5225 7900 5225
 $Comp
-L GND #PWR045
+L GND #PWR043
 U 1 1 59FD0919
 P 8200 5475
-F 0 "#PWR045" H 8200 5225 50  0001 C CNN
+F 0 "#PWR043" H 8200 5225 50  0001 C CNN
 F 1 "GND" H 8200 5325 50  0000 C CNN
 F 2 "" H 8200 5475 50  0001 C CNN
@@
 NoConn ~ 3025 4825
 $Comp
-L GND #PWR047
+L GND #PWR044
 U 1 1 5A0102F0
 P 3025 4925
-F 0 "#PWR047" H 3025 4675 50  0001 C CNN
+F 0 "#PWR044" H 3025 4675 50  0001 C CNN
 F 1 "GND" H 3025 4775 50  0000 C CNN
 F 2 "" H 3025 4925 50  0001 C CNN
@@
 $EndComp
 $Comp
-L +5V #PWR?
+L +5V #PWR045
 U 1 1 5A818AEE
 P 2750 4625
-F 0 "#PWR?" H 2750 4475 50  0001 C CNN
+F 0 "#PWR045" H 2750 4475 50  0001 C CNN
 F 1 "+5V" H 2750 4765 50  0000 C CNN
 F 2 "" H 2750 4625 50  0001 C CNN
@@
 $EndComp
 $Comp
-L +5V #PWR?
+L +5V #PWR046
 U 1 1 5A818FB4
 P 8200 4675
-F 0 "#PWR?" H 8200 4525 50  0001 C CNN
+F 0 "#PWR046" H 8200 4525 50  0001 C CNN
 F 1 "+5V" H 8200 4815 50  0000 C CNN
 F 2 "" H 8200 4675 50  0001 C CNN
@@
 $EndComp
 $Comp
-L +5V #PWR?
+L +5V #PWR047
 U 1 1 5A8195A5
 P 3850 4225
-F 0 "#PWR?" H 3850 4075 50  0001 C CNN
+F 0 "#PWR047" H 3850 4075 50  0001 C CNN
 F 1 "+5V" H 3850 4365 50  0000 C CNN
 F 2 "" H 3850 4225 50  0001 C CNN
