File: kicad/Signal_Input.sch (KiCad schematic (older format))
At the start: 30 parts, among them J2 CONN_COAXIAL, J3 CONN_COAXIAL, J4 CONN_COAXIAL, T1 WBC16-1T, T2 WBC16-1T, U10 MC12093, U11 LTC6957-3, U9 LTC6957-3

Commit message: Layout [in progress]
Connections:
- net GND: now also U11.13 (GND_Panel), U9.13 (GND_Panel)
Changed lines of the file:
@@
 $EndDescr
 $Comp
-L GND #PWR097
+L GND #PWR099
 U 1 1 595E1304
 P 3725 1675
-F 0 "#PWR097" H 3725 1425 50  0001 C CNN
+F 0 "#PWR099" H 3725 1425 50  0001 C CNN
 F 1 "GND" H 3725 1525 50  0000 C CNN
 F 2 "" H 3725 1675 50  0001 C CNN
@@
 $EndComp
 $Comp
-L GND #PWR098
+L GND #PWR0100
 U 1 1 595E15F9
 P 3175 1875
-F 0 "#PWR098" H 3175 1625 50  0001 C CNN
+F 0 "#PWR0100" H 3175 1625 50  0001 C CNN
 F 1 "GND" H 3175 1725 50  0000 C CNN
 F 2 "" H 3175 1875 50  0001 C CNN
@@
 $EndComp
 $Comp
-L GND #PWR099
+L GND #PWR0101
 U 1 1 595E4D57
 P 6325 2225
-F 0 "#PWR099" H 6325 1975 50  0001 C CNN
+F 0 "#PWR0101" H 6325 1975 50  0001 C CNN
 F 1 "GND" H 6325 2075 50  0000 C CNN
 F 2 "" H 6325 2225 50  0001 C CNN
@@
 $EndComp
 $Comp
-L GND #PWR0100
+L GND #PWR0102
 U 1 1 595E55DF
 P 6600 3900
-F 0 "#PWR0100" H 6600 3650 50  0001 C CNN
+F 0 "#PWR0102" H 6600 3650 50  0001 C CNN
 F 1 "GND" H 6600 3750 50  0000 C CNN
 F 2 "" H 6600 3900 50  0001 C CNN
@@
 $EndComp
 $Comp
-L +3.3V #PWR0101
+L +3.3V #PWR0103
 U 1 1 595E5A7F
 P 4950 3075
-F 0 "#PWR0101" H 4950 2925 50  0001 C CNN
+F 0 "#PWR0103" H 4950 2925 50  0001 C CNN
 F 1 "+3.3V" H 4950 3215 50  0000 C CNN
 F 2 "" H 4950 3075 50  0001 C CNN
@@
 $EndComp
 $Comp
-L GND #PWR0102
+L GND #PWR0104
 U 1 1 595E5BA0
 P 4950 3375
-F 0 "#PWR0102" H 4950 3125 50  0001 C CNN
+F 0 "#PWR0104" H 4950 3125 50  0001 C CNN
 F 1 "GND" H 4950 3225 50  0000 C CNN
 F 2 "" H 4950 3375 50  0001 C CNN
@@
 $EndComp
 $Comp
-L GND #PWR0103
+L GND #PWR0105
 U 1 1 595E5D32
 P 5600 4300
-F 0 "#PWR0103" H 5600 4050 50  0001 C CNN
+F 0 "#PWR0105" H 5600 4050 50  0001 C CNN
 F 1 "GND" H 5600 4150 50  0000 C CNN
 F 2 "" H 5600 4300 50  0001 C CNN
@@
 $EndComp
 $Comp
-L GND #PWR0104
+L GND #PWR0106
 U 1 1 595E6248
 P 5375 4300
-F 0 "#PWR0104" H 5375 4050 50  0001 C CNN
+F 0 "#PWR0106" H 5375 4050 50  0001 C CNN
 F 1 "GND" H 5375 4150 50  0000 C CNN
 F 2 "" H 5375 4300 50  0001 C CNN
@@
 $EndComp
 $Comp
-L GND #PWR0105
+L GND #PWR0107
 U 1 1 595E6503
 P 4250 4275
-F 0 "#PWR0105" H 4250 4025 50  0001 C CNN
+F 0 "#PWR0107" H 4250 4025 50  0001 C CNN
 F 1 "GND" H 4250 4125 50  0000 C CNN
 F 2 "" H 4250 4275 50  0001 C CNN
@@
 $EndComp
 $Comp
-L GND #PWR0106
+L GND #PWR0108
 U 1 1 595E7846
 P 2200 3925
-F 0 "#PWR0106" H 2200 3675 50  0001 C CNN
+F 0 "#PWR0108" H 2200 3675 50  0001 C CNN
 F 1 "GND" H 2200 3775 50  0000 C CNN
 F 2 "" H 2200 3925 50  0001 C CNN
@@
 Ext_Ref
 $Comp
-L GND #PWR0107
+L GND #PWR0109
 U 1 1 595E865F
 P 1900 1875
-F 0 "#PWR0107" H 1900 1625 50  0001 C CNN
+F 0 "#PWR0109" H 1900 1625 50  0001 C CNN
 F 1 "GND" H 1900 1725 50  0000 C CNN
 F 2 "" H 1900 1875 50  0001 C CNN
@@
 $EndComp
 $Comp
-L +3.3V #PWR0108
+L +3.3V #PWR0110
 U 1 1 595E9F37
 P 6050 1875
-F 0 "#PWR0108" H 6050 1725 50  0001 C CNN
+F 0 "#PWR0110" H 6050 1725 50  0001 C CNN
 F 1 "+3.3V" H 6050 2015 50  0000 C CNN
 F 2 "" H 6050 1875 50  0001 C CNN
@@
 Clk_A
 $Comp
-L +3.3V #PWR0109
+L +3.3V #PWR0111
 U 1 1 595EC3C2
 P 6800 4075
-F 0 "#PWR0109" H 6800 3925 50  0001 C CNN
+F 0 "#PWR0111" H 6800 3925 50  0001 C CNN
 F 1 "+3.3V" H 6800 4215 50  0000 C CNN
 F 2 "" H 6800 4075 50  0001 C CNN
@@
 $EndComp
 $Comp
-L GND #PWR0110
+L GND #PWR0112
 U 1 1 59655519
 P 6050 2225
-F 0 "#PWR0110" H 6050 1975 50  0001 C CNN
+F 0 "#PWR0112" H 6050 1975 50  0001 C CNN
 F 1 "GND" H 6050 2075 50  0000 C CNN
 F 2 "" H 6050 2225 50  0001 C CNN
@@
 CHA_FILTB
 $Comp
-L GND #PWR0111
+L GND #PWR0113
 U 1 1 59659874
 P 8050 2075
-F 0 "#PWR0111" H 8050 1825 50  0001 C CNN
+F 0 "#PWR0113" H 8050 1825 50  0001 C CNN
 F 1 "GND" H 8050 1925 50  0000 C CNN
 F 2 "" H 8050 2075 50  0001 C CNN
@@
 	5800 1325 5800 1600
 $Comp
-L GND #PWR0112
+L GND #PWR0114
 U 1 1 596B8167
 P 3925 5625
-F 0 "#PWR0112" H 3925 5375 50  0001 C CNN
+F 0 "#PWR0114" H 3925 5375 50  0001 C CNN
 F 1 "GND" H 3925 5475 50  0000 C CNN
 F 2 "" H 3925 5625 50  0001 C CNN
@@
 $EndComp
 $Comp
-L GND #PWR0113
+L GND #PWR0115
 U 1 1 596B8179
 P 3375 5825
-F 0 "#PWR0113" H 3375 5575 50  0001 C CNN
+F 0 "#PWR0115" H 3375 5575 50  0001 C CNN
 F 1 "GND" H 3375 5675 50  0000 C CNN
 F 2 "" H 3375 5825 50  0001 C CNN
@@
 $EndComp
 $Comp
-L GND #PWR0114
+L GND #PWR0116
 U 1 1 596B819D
 P 6525 6175
-F 0 "#PWR0114" H 6525 5925 50  0001 C CNN
+F 0 "#PWR0116" H 6525 5925 50  0001 C CNN
 F 1 "GND" H 6525 6025 50  0000 C CNN
 F 2 "" H 6525 6175 50  0001 C CNN
@@
 CH_B
 $Comp
-L GND #PWR0115
+L GND #PWR0117
 U 1 1 596B81AA
 P 2100 5825
-F 0 "#PWR0115" H 2100 5575 50  0001 C CNN
+F 0 "#PWR0117" H 2100 5575 50  0001 C CNN
 F 1 "GND" H 2100 5675 50  0000 C CNN
 F 2 "" H 2100 5825 50  0001 C CNN
@@
 $EndComp
 $Comp
-L +3.3V #PWR0116
+L +3.3V #PWR0118
 U 1 1 596B81B6
 P 6250 5825
-F 0 "#PWR0116" H 6250 5675 50  0001 C CNN
+F 0 "#PWR0118" H 6250 5675 50  0001 C CNN
 F 1 "+3.3V" H 6250 5965 50  0000 C CNN
 F 2 "" H 6250 5825 50  0001 C CNN
@@
 $EndComp
 $Comp
-L GND #PWR0117
+L GND #PWR0119
 U 1 1 596B81C4
 P 6250 6175
-F 0 "#PWR0117" H 6250 5925 50  0001 C CNN
+F 0 "#PWR0119" H 6250 5925 50  0001 C CNN
 F 1 "GND" H 6250 6025 50  0000 C CNN
 F 2 "" H 6250 6175 50  0001 C CNN
@@
 CHB_FILTB
 $Comp
-L GND #PWR0118
+L GND #PWR0120
 U 1 1 596B81CC
 P 8250 6025
-F 0 "#PWR0118" H 8250 5775 50  0001 C CNN
+F 0 "#PWR0120" H 8250 5775 50  0001 C CNN
 F 1 "GND" H 8250 5875 50  0000 C CNN
 F 2 "" H 8250 6025 50  0001 C CNN
@@
 Text Label 5800 1700 0    60   ~ 0
 IN-
+$Comp
+L GND #PWR0121
+U 1 1 596CACB7
+P 7175 2500
+F 0 "#PWR0121" H 7175 2250 50  0001 C CNN
+F 1 "GND" H 7175 2350 50  0000 C CNN
+F 2 "" H 7175 2500 50  0001 C CNN
+F 3 "" H 7175 2500 50  0001 C CNN
+	1    7175 2500
+	1    0    0    -1
+$EndComp
+$Comp
+L GND #PWR0122
+U 1 1 596CAD1C
+P 7375 6450
+F 0 "#PWR0122" H 7375 6200 50  0001 C CNN
+F 1 "GND" H 7375 6300 50  0000 C CNN
+F 2 "" H 7375 6450 50  0001 C CNN
+F 3 "" H 7375 6450 50  0001 C CNN
+	1    7375 6450
+	1    0    0    -1
+$EndComp
 $EndSCHEMATC

Commit message: layout [in progress]
Changed lines of the file:
@@
 encoding utf-8
 Sheet 5 5
-Title ""
-Date ""
-Rev ""
-Comp ""
-Comment1 ""
-Comment2 ""
+Title "FrequnecyCounter"
+Date "2017-07-19"
+Rev "01"
+Comp "COMLAB"
+Comment1 "Author: Lukas Jenni"
+Comment2 "Review: "
 Comment3 ""
 Comment4 ""
 $EndDescr
 $Comp
-L GND #PWR099
+L GND #PWR0101
 U 1 1 595E1304
 P 3725 1675
-F 0 "#PWR099" H 3725 1425 50  0001 C CNN
+F 0 "#PWR0101" H 3725 1425 50  0001 C CNN
 F 1 "GND" H 3725 1525 50  0000 C CNN
 F 2 "" H 3725 1675 50  0001 C CNN
@@
 $EndComp
 $Comp
-L GND #PWR0100
+L GND #PWR0102
 U 1 1 595E15F9
 P 3175 1875
-F 0 "#PWR0100" H 3175 1625 50  0001 C CNN
+F 0 "#PWR0102" H 3175 1625 50  0001 C CNN
 F 1 "GND" H 3175 1725 50  0000 C CNN
 F 2 "" H 3175 1875 50  0001 C CNN
@@
 $EndComp
 $Comp
-L GND #PWR0101
+L GND #PWR0103
 U 1 1 595E4D57
 P 6325 2225
-F 0 "#PWR0101" H 6325 1975 50  0001 C CNN
+F 0 "#PWR0103" H 6325 1975 50  0001 C CNN
 F 1 "GND" H 6325 2075 50  0000 C CNN
 F 2 "" H 6325 2225 50  0001 C CNN
@@
 $EndComp
 $Comp
-L GND #PWR0102
+L GND #PWR0104
 U 1 1 595E55DF
-P 6600 3900
-F 0 "#PWR0102" H 6600 3650 50  0001 C CNN
-F 1 "GND" H 6600 3750 50  0000 C CNN
-F 2 "" H 6600 3900 50  0001 C CNN
-F 3 "" H 6600 3900 50  0001 C CNN
-	1    6600 3900
+P 6600 3925
+F 0 "#PWR0104" H 6600 3675 50  0001 C CNN
+F 1 "GND" H 6600 3775 50  0000 C CNN
+F 2 "" H 6600 3925 50  0001 C CNN
+F 3 "" H 6600 3925 50  0001 C CNN
+	1    6600 3925
 	1    0    0    -1
 $EndComp
@@
 $EndComp
 $Comp
-L +3.3V #PWR0103
+L +3.3V #PWR0105
 U 1 1 595E5A7F
 P 4950 3075
-F 0 "#PWR0103" H 4950 2925 50  0001 C CNN
+F 0 "#PWR0105" H 4950 2925 50  0001 C CNN
 F 1 "+3.3V" H 4950 3215 50  0000 C CNN
 F 2 "" H 4950 3075 50  0001 C CNN
@@
 $EndComp
 $Comp
-L GND #PWR0104
+L GND #PWR0106
 U 1 1 595E5BA0
-P 4950 3375
-F 0 "#PWR0104" H 4950 3125 50  0001 C CNN
-F 1 "GND" H 4950 3225 50  0000 C CNN
-F 2 "" H 4950 3375 50  0001 C CNN
-F 3 "" H 4950 3375 50  0001 C CNN
-	1    4950 3375
-	1    0    0    -1
-$EndComp
-$Comp
-L GND #PWR0105
+P 4950 3425
+F 0 "#PWR0106" H 4950 3175 50  0001 C CNN
+F 1 "GND" H 4950 3275 50  0000 C CNN
+F 2 "" H 4950 3425 50  0001 C CNN
+F 3 "" H 4950 3425 50  0001 C CNN
+	1    4950 3425
+	1    0    0    -1
+$EndComp
+$Comp
+L GND #PWR0107
 U 1 1 595E5D32
 P 5600 4300
-F 0 "#PWR0105" H 5600 4050 50  0001 C CNN
+F 0 "#PWR0107" H 5600 4050 50  0001 C CNN
 F 1 "GND" H 5600 4150 50  0000 C CNN
 F 2 "" H 5600 4300 50  0001 C CNN
@@
 $EndComp
 $Comp
-L GND #PWR0106
+L GND #PWR0108
 U 1 1 595E6248
 P 5375 4300
-F 0 "#PWR0106" H 5375 4050 50  0001 C CNN
+F 0 "#PWR0108" H 5375 4050 50  0001 C CNN
 F 1 "GND" H 5375 4150 50  0000 C CNN
 F 2 "" H 5375 4300 50  0001 C CNN
@@
 $EndComp
 $Comp
-L GND #PWR0107
+L GND #PWR0109
 U 1 1 595E6503
 P 4250 4275
-F 0 "#PWR0107" H 4250 4025 50  0001 C CNN
+F 0 "#PWR0109" H 4250 4025 50  0001 C CNN
 F 1 "GND" H 4250 4125 50  0000 C CNN
 F 2 "" H 4250 4275 50  0001 C CNN
@@
 $EndComp
 $Comp
-L GND #PWR0108
+L GND #PWR0110
 U 1 1 595E7846
 P 2200 3925
-F 0 "#PWR0108" H 2200 3675 50  0001 C CNN
+F 0 "#PWR0110" H 2200 3675 50  0001 C CNN
 F 1 "GND" H 2200 3775 50  0000 C CNN
 F 2 "" H 2200 3925 50  0001 C CNN
@@
 Ext_Ref
 $Comp
-L GND #PWR0109
+L GND #PWR0111
 U 1 1 595E865F
 P 1900 1875
-F 0 "#PWR0109" H 1900 1625 50  0001 C CNN
+F 0 "#PWR0111" H 1900 1625 50  0001 C CNN
 F 1 "GND" H 1900 1725 50  0000 C CNN
 F 2 "" H 1900 1875 50  0001 C CNN
@@
 $EndComp
 $Comp
-L +3.3V #PWR0110
+L +3.3V #PWR0112
 U 1 1 595E9F37
 P 6050 1875
-F 0 "#PWR0110" H 6050 1725 50  0001 C CNN
+F 0 "#PWR0112" H 6050 1725 50  0001 C CNN
 F 1 "+3.3V" H 6050 2015 50  0000 C CNN
 F 2 "" H 6050 1875 50  0001 C CNN
@@
 Clk_A
 $Comp
-L +3.3V #PWR0111
+L +3.3V #PWR0113
 U 1 1 595EC3C2
 P 6800 4075
-F 0 "#PWR0111" H 6800 3925 50  0001 C CNN
+F 0 "#PWR0113" H 6800 3925 50  0001 C CNN
 F 1 "+3.3V" H 6800 4215 50  0000 C CNN
 F 2 "" H 6800 4075 50  0001 C CNN
@@
 $EndComp
 $Comp
-L GND #PWR0112
+L GND #PWR0114
 U 1 1 59655519
 P 6050 2225
-F 0 "#PWR0112" H 6050 1975 50  0001 C CNN
+F 0 "#PWR0114" H 6050 1975 50  0001 C CNN
 F 1 "GND" H 6050 2075 50  0000 C CNN
 F 2 "" H 6050 2225 50  0001 C CNN
@@
 CHA_FILTB
 $Comp
-L GND #PWR0113
+L GND #PWR0115
 U 1 1 59659874
 P 8050 2075
-F 0 "#PWR0113" H 8050 1825 50  0001 C CNN
+F 0 "#PWR0115" H 8050 1825 50  0001 C CNN
 F 1 "GND" H 8050 1925 50  0000 C CNN
 F 2 "" H 8050 2075 50  0001 C CNN
@@
 	6500 3775 6600 3775
 Wire Wire Line
-	6600 3775 6600 3900
+	6600 3775 6600 3925
 Wire Wire Line
 	6600 3900 6500 3900
@@
 	5800 1325 5800 1600
 $Comp
-L GND #PWR0114
+L GND #PWR0116
 U 1 1 596B8167
 P 3925 5625
-F 0 "#PWR0114" H 3925 5375 50  0001 C CNN
+F 0 "#PWR0116" H 3925 5375 50  0001 C CNN
 F 1 "GND" H 3925 5475 50  0000 C CNN
 F 2 "" H 3925 5625 50  0001 C CNN
@@
 $EndComp
 $Comp
-L GND #PWR0115
+L GND #PWR0117
 U 1 1 596B8179
 P 3375 5825
-F 0 "#PWR0115" H 3375 5575 50  0001 C CNN
+F 0 "#PWR0117" H 3375 5575 50  0001 C CNN
 F 1 "GND" H 3375 5675 50  0000 C CNN
 F 2 "" H 3375 5825 50  0001 C CNN
@@
 $EndComp
 $Comp
-L GND #PWR0116
+L GND #PWR0118
 U 1 1 596B819D
 P 6525 6175
-F 0 "#PWR0116" H 6525 5925 50  0001 C CNN
+F 0 "#PWR0118" H 6525 5925 50  0001 C CNN
 F 1 "GND" H 6525 6025 50  0000 C CNN
 F 2 "" H 6525 6175 50  0001 C CNN
@@
 CH_B
 $Comp
-L GND #PWR0117
+L GND #PWR0119
 U 1 1 596B81AA
 P 2100 5825
-F 0 "#PWR0117" H 2100 5575 50  0001 C CNN
+F 0 "#PWR0119" H 2100 5575 50  0001 C CNN
 F 1 "GND" H 2100 5675 50  0000 C CNN
 F 2 "" H 2100 5825 50  0001 C CNN
@@
 $EndComp
 $Comp
-L +3.3V #PWR0118
+L +3.3V #PWR0120
 U 1 1 596B81B6
 P 6250 5825
-F 0 "#PWR0118" H 6250 5675 50  0001 C CNN
+F 0 "#PWR0120" H 6250 5675 50  0001 C CNN
 F 1 "+3.3V" H 6250 5965 50  0000 C CNN
 F 2 "" H 6250 5825 50  0001 C CNN
@@
 $EndComp
 $Comp
-L GND #PWR0119
+L GND #PWR0121
 U 1 1 596B81C4
 P 6250 6175
-F 0 "#PWR0119" H 6250 5925 50  0001 C CNN
+F 0 "#PWR0121" H 6250 5925 50  0001 C CNN
 F 1 "GND" H 6250 6025 50  0000 C CNN
 F 2 "" H 6250 6175 50  0001 C CNN
@@
 CHB_FILTB
 $Comp
-L GND #PWR0120
+L GND #PWR0122
 U 1 1 596B81CC
 P 8250 6025
-F 0 "#PWR0120" H 8250 5775 50  0001 C CNN
+F 0 "#PWR0122" H 8250 5775 50  0001 C CNN
 F 1 "GND" H 8250 5875 50  0000 C CNN
 F 2 "" H 8250 6025 50  0001 C CNN
@@
 IN-
 $Comp
-L GND #PWR0121
+L GND #PWR0123
 U 1 1 596CACB7
 P 7175 2500
-F 0 "#PWR0121" H 7175 2250 50  0001 C CNN
+F 0 "#PWR0123" H 7175 2250 50  0001 C CNN
 F 1 "GND" H 7175 2350 50  0000 C CNN
 F 2 "" H 7175 2500 50  0001 C CNN
@@
 $EndComp
 $Comp
-L GND #PWR0122
+L GND #PWR0124
 U 1 1 596CAD1C
 P 7375 6450
-F 0 "#PWR0122" H 7375 6200 50  0001 C CNN
+F 0 "#PWR0124" H 7375 6200 50  0001 C CNN
 F 1 "GND" H 7375 6300 50  0000 C CNN
 F 2 "" H 7375 6450 50  0001 C CNN
@@
 	1    0    0    -1
 $EndComp
+Wire Wire Line
+	4950 3425 4950 3375
+Connection ~ 6600 3900
 $EndSCHEMATC

Commit message: Rework hardware schematic [in progress]
Parts:
- removed C50, C52, C53: 100n, Capacitors_SMD:C_0603_HandSoldering, symbol C
- removed R37: 47R, Resistors_SMD:R_0603_HandSoldering, symbol R
- removed R38: 100R, Resistors_SMD:R_0603_HandSoldering, symbol R
- removed T2: WBC16-1T, Footprints_LJ:wbc-16-1T, symbol WBC16-1T
- removed U11: LTC6957-3, Housings_DFN_QFN:DFN-12-1EP_3x3mm_Pitch0.45mm, symbol LTC6957-3
- removed V2: HSMS-281C-TR1G, TO_SOT_Packages_SMD:SOT-323_SC-70_Handsoldering, symbol HSMS-281C-TR1G
- added D3, D4: BAV99, TO_SOT_Packages_SMD:SOT-23, symbol BAV99
- added R17, R22: 680R, Resistors_SMD:R_0603_HandSoldering, symbol R
- added R23: 1k, Resistors_SMD:R_0603_HandSoldering, symbol R
- added U12: TLV3501, SMD_Packages:SOIC-8-N, symbol TLV3501
- added U13: ADR5040, TO_SOT_Packages_SMD:SOT-323_SC-70_Handsoldering, symbol ADR5040
- C51: value 100n -> 100p
- R35: value 100R -> 100k
- R36: value 560R -> 1k
Connections:
- net +3V3: now also R23.2, U12.7 (VCC)
- net CH_A: now also D3.1, D3.2
- net CH_B: now also D4.1, D4.2, U12.3 (IN+); no longer C51.2
- net Clk_A: now also C51.1, R17.2, R22.1; no longer U10.4 (OUT)
- net Clk_B: now also U12.6 (OUT)
- net GND: now also R36.2, D3.3, D4.3, R22.2, U12.4 (GND), U13.2 (V-)
- net CHB+: no longer names the net of R35.1
- net CHB+: now also R23.1, U13.1 (V+); no longer R36.1
- net T2+: no longer names the net of R35.2
- net T2+: now also R36.1, U12.2 (IN-)
- new net: C51.2, U10.4 (OUT)
- new net +1.2V: R17.1
- no-connect marks 2 -> 3
Other:
- moved on the sheet: C47, C48, C49, J3, R34, U10

Commit message: Layout changes [in progress]
Parts:
- added C50: 100n, Capacitors_SMD:C_0603_HandSoldering, symbol C
Connections:
- net +3V3: now also C50.1
- net GND: now also C50.2
Changed lines of the file:
@@
 L +3.3V #PWR0122
 U 1 1 59DC38DE
-P 5200 5975
-F 0 "#PWR0122" H 5200 5825 50  0001 C CNN
-F 1 "+3.3V" H 5200 6115 50  0000 C CNN
-F 2 "" H 5200 5975 50  0001 C CNN
-F 3 "" H 5200 5975 50  0001 C CNN
-	1    5200 5975
+P 4900 5975
+F 0 "#PWR0122" H 4900 5825 50  0001 C CNN
+F 1 "+3.3V" H 4900 6115 50  0000 C CNN
+F 2 "" H 4900 5975 50  0001 C CNN
+F 3 "" H 4900 5975 50  0001 C CNN
+	1    4900 5975
 	1    0    0    -1
 $EndComp
@@
 Wire Wire Line
 	5200 5975 5200 6000
+$Comp
+L C C50
+U 1 1 59DE4E0E
+P 4900 6125
+F 0 "C50" H 4925 6225 50  0000 L CNN
+F 1 "100n" H 4925 6025 50  0000 L CNN
+F 2 "Capacitors_SMD:C_0603_HandSoldering" H 4938 5975 50  0001 C CNN
+F 3 "" H 4900 6125 50  0001 C CNN
+	1    4900 6125
+	1    0    0    -1
+$EndComp
+Wire Wire Line
+	4900 5975 5200 5975
+$Comp
+L GND #PWR0128
+U 1 1 59DE4F7D
+P 4900 6275
+F 0 "#PWR0128" H 4900 6025 50  0001 C CNN
+F 1 "GND" H 4900 6125 50  0000 C CNN
+F 2 "" H 4900 6275 50  0001 C CNN
+F 3 "" H 4900 6275 50  0001 C CNN
+	1    4900 6275
+	1    0    0    -1
+$EndComp
 $EndSCHEMATC
