File: kicad/Signal_Input.sch (KiCad schematic (older format))
At the start: 27 parts, among them J2 CONN_COAXIAL, J3 CONN_COAXIAL, J4 CONN_COAXIAL, T1 WBC16-1T, U10 MC12093, U12 TLV3501, U9 LTC6957-3

Commit message: Small schematic and layout changes
Parts:
- added C50, C52: 100n, Capacitors_SMD:C_0603_HandSoldering, symbol C
- added R20, R3: R, Resistors_SMD:R_0603_HandSoldering, symbol R
- added R21: 100k, Resistors_SMD:R_0603_HandSoldering, symbol R
- added R23: 10k, Resistors_SMD:R_0603_HandSoldering, symbol R
- R18, R19: value 330R -> 3.3k
Connections:
- net +3V3: now also C50.1, R21.1, R3.2
- net CH_B: now also R20.2, R3.1
- net Clk_B: now also R20.1
- net GND: now also C50.2, C52.2, R23.2; no longer U10.3 (SW2), U10.6 (SW1), U12.2 (IN-)
- new net: C52.1, R21.2, R23.1, U12.2 (IN-)
- new net DIV_SW1: U10.6 (SW1)
- new net DIV_SW2: U10.3 (SW2)
Other:
- moved on the sheet: J4, R19, U12, V2

Commit message: layout commit after generating Gerberfiles
Other:
- note added: "fg = 4.68 MHz\n"
- note removed: "fg = 2.3405MHz\n"
Changed lines of the file:
@@
 	2375 3725 4200 3725
 Text Notes 6950 3325 0    60   ~ 0
-fg = 2.3405MHz\n
+fg = 4.68 MHz\n
 Text Notes 3975 3550 0    60   ~ 0
 fg = 3.183MHz\n

Commit message: Changed some component values to increase the fit & Changed power-supply of the eeprom to use the PWR_EN of the FT2232D
Parts:
- C48: value 1n -> 100p
- C51: value 100p -> 47p
- R17, R22: value 680R -> 2k
Other:
- note added: "fg = 31.83MHz\n"
- note removed: "fg = 3.183MHz\n"
Changed lines of the file:
@@
 P 4350 3725
 F 0 "C48" H 4375 3825 50  0000 L CNN
-F 1 "1n" H 4375 3625 50  0000 L CNN
+F 1 "100p" H 4375 3625 50  0000 L CNN
 F 2 "Capacitors_SMD:C_0603_HandSoldering" H 4388 3575 50  0001 C CNN
 F 3 "" H 4350 3725 50  0001 C CNN
@@
 P 7850 3775
 F 0 "R22" V 7930 3775 50  0000 C CNN
-F 1 "680R" V 7850 3775 50  0000 C CNN
+F 1 "2k" V 7850 3775 50  0000 C CNN
 F 2 "Resistors_SMD:R_0603_HandSoldering" V 7780 3775 50  0001 C CNN
 F 3 "" H 7850 3775 50  0001 C CNN
@@
 P 7850 3325
 F 0 "R17" V 7930 3325 50  0000 C CNN
-F 1 "680R" V 7850 3325 50  0000 C CNN
+F 1 "2k" V 7850 3325 50  0000 C CNN
 F 2 "Resistors_SMD:R_0603_HandSoldering" V 7780 3325 50  0001 C CNN
 F 3 "" H 7850 3325 50  0001 C CNN
@@
 P 7375 3550
 F 0 "C51" H 7400 3650 50  0000 L CNN
-F 1 "100p" H 7400 3450 50  0000 L CNN
+F 1 "47p" H 7400 3450 50  0000 L CNN
 F 2 "Capacitors_SMD:C_0603_HandSoldering" H 7413 3400 50  0001 C CNN
 F 3 "" H 7375 3550 50  0001 C CNN
@@
 fg = 4.68 MHz\n
 Text Notes 3975 3550 0    60   ~ 0
-fg = 3.183MHz\n
+fg = 31.83MHz\n
 $Comp
 L R R20

Commit message: clean up in layout & add exports (assembly drawings)
Parts:
- C43, C44, C45, C46, C47, C48, C49, C50, C51, C52: footprint Capacitors_SMD:C_0603_HandSoldering -> Footprints_LJ:Cap_0603_HandSoldering_1
Changed lines of the file:
@@
 F 0 "C43" H 5075 1425 50  0000 L CNN
 F 1 "100n" H 5075 1225 50  0000 L CNN
-F 2 "Capacitors_SMD:C_0603_HandSoldering" H 5088 1175 50  0001 C CNN
+F 2 "Footprints_LJ:Cap_0603_HandSoldering_1" H 5088 1175 50  0001 C CNN
 F 3 "" H 5050 1325 50  0001 C CNN
 	1    5050 1325
@@
 F 0 "C45" H 5075 2075 50  0000 L CNN
 F 1 "100n" H 5075 1875 50  0000 L CNN
-F 2 "Capacitors_SMD:C_0603_HandSoldering" H 5088 1825 50  0001 C CNN
+F 2 "Footprints_LJ:Cap_0603_HandSoldering_1" H 5088 1825 50  0001 C CNN
 F 3 "" H 5050 1975 50  0001 C CNN
 	1    5050 1975
@@
 F 0 "C44" H 2600 1575 50  0000 L CNN
 F 1 "100n" H 2600 1375 50  0000 L CNN
-F 2 "Capacitors_SMD:C_0603_HandSoldering" H 2613 1325 50  0001 C CNN
+F 2 "Footprints_LJ:Cap_0603_HandSoldering_1" H 2613 1325 50  0001 C CNN
 F 3 "" H 2575 1475 50  0001 C CNN
 	1    2575 1475
@@
 F 0 "C47" H 4925 3325 50  0000 L CNN
 F 1 "100n" H 4925 3125 50  0000 L CNN
-F 2 "Capacitors_SMD:C_0603_HandSoldering" H 4938 3075 50  0001 C CNN
+F 2 "Footprints_LJ:Cap_0603_HandSoldering_1" H 4938 3075 50  0001 C CNN
 F 3 "" H 4900 3225 50  0001 C CNN
 	1    4900 3225
@@
 F 0 "C49" H 5350 4225 50  0000 L CNN
 F 1 "1n" H 5350 4025 50  0000 L CNN
-F 2 "Capacitors_SMD:C_0603_HandSoldering" H 5363 3975 50  0001 C CNN
+F 2 "Footprints_LJ:Cap_0603_HandSoldering_1" H 5363 3975 50  0001 C CNN
 F 3 "" H 5325 4125 50  0001 C CNN
 	1    5325 4125
@@
 F 0 "C48" H 4375 3825 50  0000 L CNN
 F 1 "100p" H 4375 3625 50  0000 L CNN
-F 2 "Capacitors_SMD:C_0603_HandSoldering" H 4388 3575 50  0001 C CNN
+F 2 "Footprints_LJ:Cap_0603_HandSoldering_1" H 4388 3575 50  0001 C CNN
 F 3 "" H 4350 3725 50  0001 C CNN
 	1    4350 3725
@@
 F 0 "C46" H 5750 2125 50  0000 L CNN
 F 1 "100n" H 5750 1925 50  0000 L CNN
-F 2 "Capacitors_SMD:C_0603_HandSoldering" H 5763 1875 50  0001 C CNN
+F 2 "Footprints_LJ:Cap_0603_HandSoldering_1" H 5763 1875 50  0001 C CNN
 F 3 "" H 5725 2025 50  0001 C CNN
 	1    5725 2025
@@
 F 0 "C51" H 7400 3650 50  0000 L CNN
 F 1 "47p" H 7400 3450 50  0000 L CNN
-F 2 "Capacitors_SMD:C_0603_HandSoldering" H 7413 3400 50  0001 C CNN
+F 2 "Footprints_LJ:Cap_0603_HandSoldering_1" H 7413 3400 50  0001 C CNN
 F 3 "" H 7375 3550 50  0001 C CNN
 	1    7375 3550
@@
 F 0 "C52" H 4000 7025 50  0000 L CNN
 F 1 "100n" H 4000 6825 50  0000 L CNN
-F 2 "Capacitors_SMD:C_0603_HandSoldering" H 4013 6775 50  0001 C CNN
+F 2 "Footprints_LJ:Cap_0603_HandSoldering_1" H 4013 6775 50  0001 C CNN
 F 3 "" H 3975 6925 50  0001 C CNN
 	1    3975 6925
@@
 F 0 "C50" H 4875 6075 50  0000 L CNN
 F 1 "100n" H 4875 5875 50  0000 L CNN
-F 2 "Capacitors_SMD:C_0603_HandSoldering" H 4888 5825 50  0001 C CNN
+F 2 "Footprints_LJ:Cap_0603_HandSoldering_1" H 4888 5825 50  0001 C CNN
 F 3 "" H 4850 5975 50  0001 C CNN
 	1    4850 5975
