File: kicad/FrequnecyCounter.sch (KiCad schematic (older format))
At the start: 0 parts

Commit message: Layout [in progress]
Parts:
- added MK1, MK2, MK3, MK4: Mounting_Hole, Mounting_Holes:MountingHole_3.2mm_M3_ISO7380, symbol Mounting_Hole
Changed lines of the file:
@@
 F0 "USB_JTAG" 60
 F1 "USB_JTAG.sch" 60
-F2 "TCK" O R 2475 1225 60
-F3 "TDI" I R 2475 1725 60
-F4 "TDO" O R 2475 1475 60
-F5 "TMS" O R 2475 1975 60
-F6 "~RESET" I L 1525 1625 60
-F7 "TXD" O R 2475 2375 60
-F8 "RXD" I R 2475 2600 60
+F2 "~RESET" I L 1525 1625 60
+F3 "TXD" O R 2475 2375 60
+F4 "RXD" I R 2475 2600 60
+F5 "TCK_FT" O R 2475 1225 60
+F6 "TDI_FT" I R 2475 1475 60
+F7 "TDO_FT" O R 2475 1725 60
+F8 "TMS_FT" O R 2475 1975 60
 $EndSheet
 $Sheet
@@
 Wire Wire Line
 	3025 5325 5650 5325
+$Comp
+L Mounting_Hole MK1
+U 1 1 596D53D7
+P 1050 7250
+F 0 "MK1" H 1050 7450 50  0000 C CNN
+F 1 "Mounting_Hole" H 1050 7375 50  0000 C CNN
+F 2 "Mounting_Holes:MountingHole_3.2mm_M3_ISO7380" H 1050 7250 50  0001 C CNN
+F 3 "" H 1050 7250 50  0001 C CNN
+	1    1050 7250
+	1    0    0    -1
+$EndComp
+$Comp
+L Mounting_Hole MK3
+U 1 1 596D5D24
+P 1050 7575
+F 0 "MK3" H 1050 7775 50  0000 C CNN
+F 1 "Mounting_Hole" H 1050 7700 50  0000 C CNN
+F 2 "Mounting_Holes:MountingHole_3.2mm_M3_ISO7380" H 1050 7575 50  0001 C CNN
+F 3 "" H 1050 7575 50  0001 C CNN
+	1    1050 7575
+	1    0    0    -1
+$EndComp
+$Comp
+L Mounting_Hole MK2
+U 1 1 596D626D
+P 1600 7250
+F 0 "MK2" H 1600 7450 50  0000 C CNN
+F 1 "Mounting_Hole" H 1600 7375 50  0000 C CNN
+F 2 "Mounting_Holes:MountingHole_3.2mm_M3_ISO7380" H 1600 7250 50  0001 C CNN
+F 3 "" H 1600 7250 50  0001 C CNN
+	1    1600 7250
+	1    0    0    -1
+$EndComp
+$Comp
+L Mounting_Hole MK4
+U 1 1 596D6346
+P 1600 7575
+F 0 "MK4" H 1600 7775 50  0000 C CNN
+F 1 "Mounting_Hole" H 1600 7700 50  0000 C CNN
+F 2 "Mounting_Holes:MountingHole_3.2mm_M3_ISO7380" H 1600 7575 50  0001 C CNN
+F 3 "" H 1600 7575 50  0001 C CNN
+	1    1600 7575
+	1    0    0    -1
+$EndComp
 $EndSCHEMATC

Commit message: Reworked schematic and layout [to review]
Changed lines of the file:
@@
-$EndSheet
-$Sheet
-S 5650 3075 1725 2800
-U 595E0A92
-F0 "FPGA" 60
-F1 "FPGA.sch" 60
-F2 "Ext_Ref_Clk" I L 5650 3275 60
-F3 "Clk_A" I L 5650 3550 60
-F4 "Clk_B" I L 5650 3800 60
-F5 "EN_CHA_FILTA" O R 7375 3275 60
-F6 "EN_CHA_FILTB" O R 7375 3525 60
-F7 "EN_CHB_FILTA" O R 7375 3775 60
-F8 "EN_CHB_FILTB" O R 7375 4025 60
-F9 "TCK" I L 5650 4050 60
-F10 "TDI" I L 5650 4300 60
-F11 "TDO" O L 5650 4575 60
-F12 "TMS" I L 5650 4825 60
-F13 "RXD" I L 5650 5100 60
-F14 "TXD" O L 5650 5325 60
 $EndSheet
 $Sheet
@@
 F8 "TMS_FT" O R 2475 1975 60
 $EndSheet
-$Sheet
-S 8325 3075 1725 1950
-U 595DF15C
-F0 "Signal_Input" 60
-F1 "Signal_Input.sch" 60
-F2 "Ext_Ref_Clk" O R 10050 3250 60
-F3 "Clk_A" O R 10050 3475 60
-F4 "Clk_B" O R 10050 3725 60
-F5 "CHA_FILTA" I L 8325 3275 60
-F6 "CHA_FILTB" I L 8325 3525 60
-F7 "CHB_FILTA" I L 8325 3775 60
-F8 "CHB_FILTB" I L 8325 4025 60
-$EndSheet
-Wire Wire Line
-	7375 4025 8325 4025
-Wire Wire Line
-	7375 3775 8325 3775
-Wire Wire Line
-	7375 3525 8325 3525
-Wire Wire Line
-	7375 3275 8325 3275
 Wire Wire Line
 	5650 3275 5200 3275
@@
 	1    0    0    -1
 $EndComp
+$Sheet
+S 8325 3075 1725 1950
+U 595DF15C
+F0 "Signal_Input" 60
+F1 "Signal_Input.sch" 60
+F2 "Ext_Ref_Clk" O R 10050 3250 60
+F3 "Clk_A" O R 10050 3475 60
+F4 "Clk_B" O R 10050 3725 60
+F5 "EXTREF_FILTA" I L 8325 3400 60
+F6 "EXTREF_FILTB" I L 8325 3600 60
+$EndSheet
+$Sheet
+S 5650 3075 1725 2800
+U 595E0A92
+F0 "FPGA" 60
+F1 "FPGA.sch" 60
+F2 "Ext_Ref_Clk" I L 5650 3275 60
+F3 "Clk_A" I L 5650 3550 60
+F4 "Clk_B" I L 5650 3800 60
+F5 "TCK" I L 5650 4050 60
+F6 "TDI" I L 5650 4300 60
+F7 "TDO" O L 5650 4575 60
+F8 "TMS" I L 5650 4825 60
+F9 "RXD" I L 5650 5100 60
+F10 "TXD" O L 5650 5325 60
+F11 "EN_EXTREF_FILTA" O R 7375 3400 60
+F12 "EN_EXTREF_FILTB" O R 7375 3600 60
+$EndSheet
+Wire Wire Line
+	8325 3600 7375 3600
+Wire Wire Line
+	7375 3400 8325 3400
 $EndSCHEMATC

Commit message: some small schematic and layout changes [completed]
Changed lines of the file:
@@
 	3650 4825 5650 4825
 Wire Wire Line
-	1200 1625 1200 3775
+	1200 1625 1200 5625
 Wire Wire Line
 	1200 3775 1525 3775
@@
 F11 "EN_EXTREF_FILTA" O R 7375 3400 60
 F12 "EN_EXTREF_FILTB" O R 7375 3600 60
+F13 "~RESET" I L 5650 5625 60
 $EndSheet
 Wire Wire Line
@@
 Wire Wire Line
 	7375 3400 8325 3400
+Connection ~ 1200 3775
+Wire Wire Line
+	1200 5625 5650 5625
 $EndSCHEMATC

Commit message: Small schematic and layout changes
Changed lines of the file:
@@
 F0 "Power_Supply" 60
 F1 "Power_Supply.sch" 60
-F2 "~RESET" O L 1525 3775 60
+F2 "~RESET" I L 1525 3775 60
 $EndSheet
 $Sheet
@@
 F0 "USB_JTAG" 60
 F1 "USB_JTAG.sch" 60
-F2 "~RESET" I L 1525 1625 60
-F3 "TXD" O R 2475 2375 60
-F4 "RXD" I R 2475 2600 60
-F5 "TCK_FT" O R 2475 1225 60
-F6 "TDI_FT" I R 2475 1475 60
-F7 "TDO_FT" O R 2475 1725 60
-F8 "TMS_FT" O R 2475 1975 60
+F2 "TXD" O R 2475 2375 60
+F3 "RXD" I R 2475 2600 60
+F4 "TCK_FT" O R 2475 1225 60
+F5 "TDI_FT" I R 2475 1475 60
+F6 "TDO_FT" O R 2475 1725 60
+F7 "TMS_FT" O R 2475 1975 60
+F8 "~RESET" O L 1525 1625 60
 $EndSheet
 Wire Wire Line
@@
 Wire Wire Line
 	3650 4825 5650 4825
-Wire Wire Line
-	1200 1625 1200 5625
 Wire Wire Line
 	1200 3775 1525 3775
@@
 F5 "EXTREF_FILTA" I L 8325 3400 60
 F6 "EXTREF_FILTB" I L 8325 3600 60
+F7 "DIV_SW2" I L 8325 4050 60
+F8 "DIV_SW1" I L 8325 4175 60
 $EndSheet
 $Sheet
@@
 F11 "EN_EXTREF_FILTA" O R 7375 3400 60
 F12 "EN_EXTREF_FILTB" O R 7375 3600 60
-F13 "~RESET" I L 5650 5625 60
+F13 "DIV_SW1" O R 7375 4175 60
+F14 "DIV_SW2" O R 7375 4050 60
 $EndSheet
 Wire Wire Line
@@
 Wire Wire Line
 	7375 3400 8325 3400
-Connection ~ 1200 3775
 Wire Wire Line
-	1200 5625 5650 5625
+	1200 3775 1200 1625
+Wire Wire Line
+	7375 4175 8325 4175
+Wire Wire Line
+	8325 4050 7375 4050
 $EndSCHEMATC
