File: kicad/Power_Supply.sch (KiCad schematic (older format))
At the start: 23 parts, among them SW1 SW_Push, U1 TPS650250, U2 LP3871

Commit message: layout [in progress]
Parts:
- R7: value 33k -> 22k
Connections:
- net labels added: +3V3_FPGA, +3V6
- net labels removed: +2V5, +3.6V
- wire segments 46 -> 58
Other:
- moved on the sheet: C10, SW1
Changed lines of the file:
@@
 encoding utf-8
 Sheet 2 5
-Title ""
-Date ""
-Rev ""
-Comp ""
-Comment1 ""
-Comment2 ""
+Title "FrequnecyCounter"
+Date "2017-07-19"
+Rev "01"
+Comp "COMLAB"
+Comment1 "Author: Lukas Jenni"
+Comment2 "Review: "
 Comment3 ""
 Comment4 ""
@@
 	4650 2625 5950 2625
 Wire Wire Line
-	5950 2625 5950 1525
-Wire Wire Line
-	5950 1525 6850 1525
-Wire Wire Line
-	6850 1525 6850 1925
-$Comp
-L C C3
-U 1 1 595D41B6
-P 6200 1675
-F 0 "C3" H 6225 1775 50  0000 L CNN
-F 1 "10u" H 6225 1575 50  0000 L CNN
-F 2 "Capacitors_SMD:C_0603_HandSoldering" H 6238 1525 50  0001 C CNN
-F 3 "" H 6200 1675 50  0001 C CNN
-	1    6200 1675
-	1    0    0    -1
-$EndComp
+	5950 2625 5950 1500
 $Comp
 L C C4
@@
 	1    0    0    -1
 $EndComp
-Text GLabel 6850 1525 2    60   UnSpc ~ 0
-+3.6V
-Text GLabel 7975 5200 0    60   UnSpc ~ 0
-+3.6V
 $Comp
 L GND #PWR08
@@
 L GND #PWR09
 U 1 1 595D5BC0
-P 10075 5500
-F 0 "#PWR09" H 10075 5250 50  0001 C CNN
-F 1 "GND" H 10075 5350 50  0000 C CNN
-F 2 "" H 10075 5500 50  0001 C CNN
-F 3 "" H 10075 5500 50  0001 C CNN
-	1    10075 5500
-	1    0    0    -1
-$EndComp
-Wire Wire Line
-	9625 5275 9700 5275
-Wire Wire Line
-	9700 5275 9700 5200
-Wire Wire Line
-	9700 5200 10250 5200
+P 10075 5550
+F 0 "#PWR09" H 10075 5300 50  0001 C CNN
+F 1 "GND" H 10075 5400 50  0000 C CNN
+F 2 "" H 10075 5550 50  0001 C CNN
+F 3 "" H 10075 5550 50  0001 C CNN
+	1    10075 5550
+	1    0    0    -1
+$EndComp
 $Comp
 L C C10
 U 1 1 595D5B10
-P 10075 5350
-F 0 "C10" H 10100 5450 50  0000 L CNN
-F 1 "10u" H 10100 5250 50  0000 L CNN
-F 2 "Capacitors_SMD:C_0603_HandSoldering" H 10113 5200 50  0001 C CNN
-F 3 "" H 10075 5350 50  0001 C CNN
-	1    10075 5350
-	1    0    0    -1
-$EndComp
-Wire Wire Line
-	7975 5200 8525 5200
-Wire Wire Line
-	8525 5200 8525 5275
-Wire Wire Line
-	8525 5275 8600 5275
+P 10075 5375
+F 0 "C10" H 10100 5475 50  0000 L CNN
+F 1 "10u" H 10100 5275 50  0000 L CNN
+F 2 "Capacitors_SMD:C_0603_HandSoldering" H 10113 5225 50  0001 C CNN
+F 3 "" H 10075 5375 50  0001 C CNN
+	1    10075 5375
+	1    0    0    -1
+$EndComp
 Wire Wire Line
 	8400 5500 8600 5500
@@
 	1    0    0    -1
 $EndComp
-Connection ~ 8400 5200
-$Comp
-L C C9
-U 1 1 595D6E13
-P 8175 5350
-F 0 "C9" H 8200 5450 50  0000 L CNN
-F 1 "10u" H 8200 5250 50  0000 L CNN
-F 2 "Capacitors_SMD:C_0603_HandSoldering" H 8213 5200 50  0001 C CNN
-F 3 "" H 8175 5350 50  0001 C CNN
-	1    8175 5350
-	1    0    0    -1
-$EndComp
 $Comp
 L GND #PWR011
@@
 L +3.3V #PWR012
 U 1 1 595D6EDC
-P 10250 5200
-F 0 "#PWR012" H 10250 5050 50  0001 C CNN
-F 1 "+3.3V" H 10250 5340 50  0000 C CNN
-F 2 "" H 10250 5200 50  0001 C CNN
-F 3 "" H 10250 5200 50  0001 C CNN
-	1    10250 5200
+P 10075 5150
+F 0 "#PWR012" H 10075 5000 50  0001 C CNN
+F 1 "+3.3V" H 10075 5290 50  0000 C CNN
+F 2 "" H 10075 5150 50  0001 C CNN
+F 3 "" H 10075 5150 50  0001 C CNN
+	1    10075 5150
 	1    0    0    -1
 $EndComp
@@
 P 8600 2925
 F 0 "R7" V 8680 2925 50  0000 C CNN
-F 1 "33k" V 8600 2925 50  0000 C CNN
+F 1 "22k" V 8600 2925 50  0000 C CNN
 F 2 "Resistors_SMD:R_0603_HandSoldering" V 8530 2925 50  0001 C CNN
 F 3 "" H 8600 2925 50  0001 C CNN
@@
 Wire Wire Line
 	2100 3675 2100 4125
-Connection ~ 6550 1525
-Connection ~ 6200 1525
 Connection ~ 5350 1175
 Connection ~ 5000 1175
@@
 NoConn ~ 4350 3725
 NoConn ~ 4350 3625
-Connection ~ 10075 5200
-Connection ~ 8175 5200
 Connection ~ 5650 1175
 $Comp
 L SW_Push SW1
 U 1 1 59642ABE
-P 1275 3475
-F 0 "SW1" H 1325 3575 50  0000 L CNN
-F 1 "SW_Push" H 1275 3415 50  0000 C CNN
-F 2 "Footprints_LJ:Mini-Taster-4pin" H 1275 3675 50  0001 C CNN
-F 3 "" H 1275 3675 50  0001 C CNN
-	1    1275 3475
+P 1275 3500
+F 0 "SW1" H 1325 3600 50  0000 L CNN
+F 1 "SW_Push" H 1275 3440 50  0000 C CNN
+F 2 "Footprints_LJ:Mini-Taster-4pin" H 1275 3700 50  0001 C CNN
+F 3 "" H 1275 3700 50  0001 C CNN
+	1    1275 3500
 	0    1    1    0
 $EndComp
@@
 L GND #PWR019
 U 1 1 596437E6
-P 1275 3675
-F 0 "#PWR019" H 1275 3425 50  0001 C CNN
-F 1 "GND" H 1275 3525 50  0000 C CNN
-F 2 "" H 1275 3675 50  0001 C CNN
-F 3 "" H 1275 3675 50  0001 C CNN
-	1    1275 3675
+P 1275 3725
+F 0 "#PWR019" H 1275 3475 50  0001 C CNN
+F 1 "GND" H 1275 3575 50  0000 C CNN
+F 2 "" H 1275 3725 50  0001 C CNN
+F 3 "" H 1275 3725 50  0001 C CNN
+	1    1275 3725
 	1    0    0    -1
 $EndComp
@@
 	1275 3275 2100 3275
 Wire Wire Line
-	1275 2275 1275 3275
+	1275 2275 1275 3300
 Wire Wire Line
 	1050 2925 2100 2925
@@
 L +5V #PWR020
 U 1 1 5964FB81
-P 1275 1975
-F 0 "#PWR020" H 1275 1825 50  0001 C CNN
-F 1 "+5V" H 1275 2115 50  0000 C CNN
-F 2 "" H 1275 1975 50  0001 C CNN
-F 3 "" H 1275 1975 50  0001 C CNN
-	1    1275 1975
-	1    0    0    -1
-$EndComp
-Wire Wire Line
-	2100 1950 2100 3525
-Connection ~ 2100 2425
-Connection ~ 2100 2775
-Connection ~ 2100 3125
+P 1275 1950
+F 0 "#PWR020" H 1275 1800 50  0001 C CNN
+F 1 "+5V" H 1275 2090 50  0000 C CNN
+F 2 "" H 1275 1950 50  0001 C CNN
+F 3 "" H 1275 1950 50  0001 C CNN
+	1    1275 1950
+	1    0    0    -1
+$EndComp
 $Comp
 L C C7
@@
 L +5V #PWR021
 U 1 1 59650E00
-P 1750 1950
-F 0 "#PWR021" H 1750 1800 50  0001 C CNN
-F 1 "+5V" H 1750 2090 50  0000 C CNN
-F 2 "" H 1750 1950 50  0001 C CNN
-F 3 "" H 1750 1950 50  0001 C CNN
-	1    1750 1950
-	1    0    0    -1
-$EndComp
-Wire Wire Line
-	1750 1950 2100 1950
-Connection ~ 2100 2275
+P 1750 1900
+F 0 "#PWR021" H 1750 1750 50  0001 C CNN
+F 1 "+5V" H 1750 2040 50  0000 C CNN
+F 2 "" H 1750 1900 50  0001 C CNN
+F 3 "" H 1750 1900 50  0001 C CNN
+	1    1750 1900
+	1    0    0    -1
+$EndComp
 $Comp
 L GND #PWR022
@@
 	1    0    0    -1
 $EndComp
-$Comp
-L +2V5 #PWR023
-U 1 1 59663D71
+Connection ~ 8600 1875
+NoConn ~ 4350 3375
+NoConn ~ 4350 3475
+Connection ~ 2100 3975
+Connection ~ 2100 3825
+$Comp
+L +3V3_FPGA #PWR023
+U 1 1 5971CBE5
 P 8600 1825
 F 0 "#PWR023" H 8600 1675 50  0001 C CNN
-F 1 "+2V5" H 8600 1965 50  0000 C CNN
+F 1 "+3V3_FPGA" H 8600 1965 50  0000 C CNN
 F 2 "" H 8600 1825 50  0001 C CNN
 F 3 "" H 8600 1825 50  0001 C CNN
@@
 	1    0    0    -1
 $EndComp
-Connection ~ 1750 1950
-Connection ~ 8600 1875
-NoConn ~ 4350 3375
+$Comp
+L +3V6 #PWR024
+U 1 1 597219FA
+P 6850 1475
+F 0 "#PWR024" H 6850 1325 50  0001 C CNN
+F 1 "+3V6" H 6850 1615 50  0000 C CNN
+F 2 "" H 6850 1475 50  0001 C CNN
+F 3 "" H 6850 1475 50  0001 C CNN
+	1    6850 1475
+	1    0    0    -1
+$EndComp
+$Comp
+L C C9
+U 1 1 595D6E13
+P 8175 5350
+F 0 "C9" H 8200 5450 50  0000 L CNN
+F 1 "10u" H 8200 5250 50  0000 L CNN
+F 2 "Capacitors_SMD:C_0603_HandSoldering" H 8213 5200 50  0001 C CNN
+F 3 "" H 8175 5350 50  0001 C CNN
+	1    8175 5350
+	1    0    0    -1
+$EndComp
+$Comp
+L C C3
+U 1 1 595D41B6
+P 6200 1675
+F 0 "C3" H 6225 1775 50  0000 L CNN
+F 1 "10u" H 6225 1575 50  0000 L CNN
+F 2 "Capacitors_SMD:C_0603_HandSoldering" H 6238 1525 50  0001 C CNN
+F 3 "" H 6200 1675 50  0001 C CNN
+	1    6200 1675
+	1    0    0    -1
+$EndComp
+Wire Wire Line
+	6850 1475 6850 1925
+Wire Wire Line
+	10075 5150 10075 5225
+Wire Wire Line
+	10075 5200 9625 5200
+Wire Wire Line
+	9625 5200 9625 5275
+Wire Wire Line
+	5950 1500 6850 1500
+Wire Wire Line
+	6200 1500 6200 1525
+Wire Wire Line
+	6550 1500 6550 1525
+Connection ~ 6200 1500
+Connection ~ 6550 1500
+Connection ~ 6850 1500
+Wire Wire Line
+	1275 1950 1275 1975
+Wire Wire Line
+	8400 5175 8400 5200
+Wire Wire Line
+	8600 5175 8600 5275
+$Comp
+L +3V6 #PWR025
+U 1 1 5977DEC2
+P 8175 5150
+F 0 "#PWR025" H 8175 5000 50  0001 C CNN
+F 1 "+3V6" H 8175 5290 50  0000 C CNN
+F 2 "" H 8175 5150 50  0001 C CNN
+F 3 "" H 8175 5150 50  0001 C CNN
+	1    8175 5150
+	1    0    0    -1
+$EndComp
+Wire Wire Line
+	8175 5150 8175 5200
+Wire Wire Line
+	8175 5175 8600 5175
+Connection ~ 8175 5175
+Connection ~ 8400 5175
 $Comp
 L TPS650250 U1
@@
 	1    0    0    -1
 $EndComp
-NoConn ~ 4350 3475
-Connection ~ 2100 3975
-Connection ~ 2100 3825
+Wire Wire Line
+	2050 3125 2100 3125
+Wire Wire Line
+	2050 2775 2100 2775
+Wire Wire Line
+	2050 2425 2100 2425
+Connection ~ 2050 2775
+Wire Wire Line
+	2050 2275 2100 2275
+Connection ~ 2050 2425
+Wire Wire Line
+	1750 1925 2050 1925
+Connection ~ 2050 2275
+Wire Wire Line
+	1750 1900 1750 1950
+Connection ~ 1750 1925
+Connection ~ 1275 3275
+Wire Wire Line
+	1275 3725 1275 3700
+Wire Wire Line
+	2050 1925 2050 3525
+Wire Wire Line
+	10075 5550 10075 5525
+Connection ~ 10075 5200
+Wire Wire Line
+	2050 3525 2100 3525
+Connection ~ 2050 3125
 $EndSCHEMATC

Commit message: Rework hardware schematic [in progress]
Connections:
- net +1.2V: now also U1.1 (VDCDC3); no longer U1.8 (VDCDC1)
- net +3V3_FPGA: now also U1.25 (VDCDC2); no longer U1.1 (VDCDC3)
- net +3V6: now also U1.8 (VDCDC1); no longer U1.25 (VDCDC2)
- net at R2.2, R6.1: now also U1.9 (DEFDCDC1); no longer U1.22 (DEFDCDC2)
- net at U1.27 (L2): now also L3.1; no longer L2.1
- net at U1.3 (L3): now also L1.1; no longer L3.1
- net at R5.2, R7.1: now also U1.22 (DEFDCDC2); no longer U1.32 (DEFDCDC3)
- net at U1.6 (L1): now also L2.1; no longer L1.1
- net at R1.2, R4.1: now also U1.32 (DEFDCDC3); no longer U1.9 (DEFDCDC1)
Other:
- moved on the sheet: C1, C2, C3, C4, C5, C6, L1, L2, L3, R1, R2, R4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

Commit message: Reworked schematic and layout [to review]
Changed lines of the file:
@@
 L GND #PWR08
 U 1 1 595D5A7A
-P 9100 5800
-F 0 "#PWR08" H 9100 5550 50  0001 C CNN
-F 1 "GND" H 9100 5650 50  0000 C CNN
-F 2 "" H 9100 5800 50  0001 C CNN
-F 3 "" H 9100 5800 50  0001 C CNN
-	1    9100 5800
+P 9100 5825
+F 0 "#PWR08" H 9100 5575 50  0001 C CNN
+F 1 "GND" H 9100 5675 50  0000 C CNN
+F 2 "" H 9100 5825 50  0001 C CNN
+F 3 "" H 9100 5825 50  0001 C CNN
+	1    9100 5825
 	1    0    0    -1
 $EndComp
@@
 L GND #PWR010
 U 1 1 595D677C
-P 9625 5500
-F 0 "#PWR010" H 9625 5250 50  0001 C CNN
-F 1 "GND" H 9625 5350 50  0000 C CNN
-F 2 "" H 9625 5500 50  0001 C CNN
-F 3 "" H 9625 5500 50  0001 C CNN
-	1    9625 5500
+P 9625 5525
+F 0 "#PWR010" H 9625 5275 50  0001 C CNN
+F 1 "GND" H 9625 5375 50  0000 C CNN
+F 2 "" H 9625 5525 50  0001 C CNN
+F 3 "" H 9625 5525 50  0001 C CNN
+	1    9625 5525
 	1    0    0    -1
 $EndComp
@@
 L GND #PWR011
 U 1 1 595D6E7D
-P 8175 5500
-F 0 "#PWR011" H 8175 5250 50  0001 C CNN
-F 1 "GND" H 8175 5350 50  0000 C CNN
-F 2 "" H 8175 5500 50  0001 C CNN
-F 3 "" H 8175 5500 50  0001 C CNN
-	1    8175 5500
+P 8175 5525
+F 0 "#PWR011" H 8175 5275 50  0001 C CNN
+F 1 "GND" H 8175 5375 50  0000 C CNN
+F 2 "" H 8175 5525 50  0001 C CNN
+F 3 "" H 8175 5525 50  0001 C CNN
+	1    8175 5525
 	1    0    0    -1
 $EndComp
@@
 Wire Wire Line
 	4650 2275 4975 2275
+Wire Wire Line
+	8175 5525 8175 5500
+Wire Wire Line
+	9625 5525 9625 5500
+Wire Wire Line
+	9100 5825 9100 5800
 $EndSCHEMATC

Commit message: Remove design errors and changes some footprints [to review]
Connections:
- net GND: now also U1.33 (GND_PANEL)
Changed lines of the file:
@@
 Wire Wire Line
 	9100 5825 9100 5800
+$Comp
+L GND #PWR026
+U 1 1 59E1CD41
+P 3150 5025
+F 0 "#PWR026" H 3150 4775 50  0001 C CNN
+F 1 "GND" H 3150 4875 50  0000 C CNN
+F 2 "" H 3150 5025 50  0001 C CNN
+F 3 "" H 3150 5025 50  0001 C CNN
+	1    3150 5025
+	1    0    0    -1
+$EndComp
 $EndSCHEMATC

Commit message: Small layout and schematic changes
Parts:
- SW1: symbol SW_Push -> SW_Push-RESCUE-FrequnecyCounter
Connections:
- net GND: now also SW1.4; no longer SW1.2
Changed lines of the file:
@@
 EESchema Schematic File Version 2
+LIBS:FrequnecyCounter-rescue
 LIBS:power
 LIBS:device
@@
 Connection ~ 8825 1875
 $Comp
-L SW_Push SW1
+L SW_Push-RESCUE-FrequnecyCounter SW1
 U 1 1 59642ABE
 P 1275 3500
+AR Path="/59642ABE" Ref="SW1"  Part="1"
+AR Path="/595D114F/59642ABE" Ref="SW1"  Part="1"
 F 0 "SW1" H 1325 3600 50  0000 L CNN
 F 1 "SW_Push" H 1275 3440 50  0000 C CNN

Commit message: Small schematic and layout changes
Parts:
- removed R3: 10k, Resistors_SMD:R_0603_HandSoldering, symbol R
- removed SW1: SW_Push, Footprints_LJ:Mini-Taster-4pin, symbol SW_Push-RESCUE-FrequnecyCounter
Changed lines of the file:
@@
 NoConn ~ 4350 3625
 Connection ~ 8825 1875
-$Comp
-L SW_Push-RESCUE-FrequnecyCounter SW1
-U 1 1 59642ABE
-P 1275 3500
-AR Path="/59642ABE" Ref="SW1"  Part="1"
-AR Path="/595D114F/59642ABE" Ref="SW1"  Part="1"
-F 0 "SW1" H 1325 3600 50  0000 L CNN
-F 1 "SW_Push" H 1275 3440 50  0000 C CNN
-F 2 "Footprints_LJ:Mini-Taster-4pin" H 1275 3700 50  0001 C CNN
-F 3 "" H 1275 3700 50  0001 C CNN
-	1    1275 3500
-	0    1    1    0
-$EndComp
-$Comp
-L GND #PWR019
-U 1 1 596437E6
-P 1275 3725
-F 0 "#PWR019" H 1275 3475 50  0001 C CNN
-F 1 "GND" H 1275 3575 50  0000 C CNN
-F 2 "" H 1275 3725 50  0001 C CNN
-F 3 "" H 1275 3725 50  0001 C CNN
-	1    1275 3725
-	1    0    0    -1
-$EndComp
 Wire Wire Line
 	1275 3275 2100 3275
-Wire Wire Line
-	1275 2275 1275 3300
 Wire Wire Line
 	1050 2925 2100 2925
@@
 	2100 2575 1275 2575
 Connection ~ 1275 2925
-Connection ~ 1275 2575
-$Comp
-L R R3
-U 1 1 59645345
-P 1275 2125
-F 0 "R3" V 1355 2125 50  0000 C CNN
-F 1 "10k" V 1275 2125 50  0000 C CNN
-F 2 "Resistors_SMD:R_0603_HandSoldering" V 1205 2125 50  0001 C CNN
-F 3 "" H 1275 2125 50  0001 C CNN
-	1    1275 2125
-	1    0    0    -1
-$EndComp
-Text HLabel 1050 2925 0    60   Output ~ 0
+Text HLabel 1050 2925 0    60   Input ~ 0
 ~RESET
-$Comp
-L +5V #PWR020
-U 1 1 5964FB81
-P 1275 1950
-F 0 "#PWR020" H 1275 1800 50  0001 C CNN
-F 1 "+5V" H 1275 2090 50  0000 C CNN
-F 2 "" H 1275 1950 50  0001 C CNN
-F 3 "" H 1275 1950 50  0001 C CNN
-	1    1275 1950
-	1    0    0    -1
-$EndComp
 $Comp
 L C C7
@@
 $EndComp
 $Comp
-L +5V #PWR021
+L +5V #PWR019
 U 1 1 59650E00
 P 1750 1900
-F 0 "#PWR021" H 1750 1750 50  0001 C CNN
+F 0 "#PWR019" H 1750 1750 50  0001 C CNN
 F 1 "+5V" H 1750 2040 50  0000 C CNN
 F 2 "" H 1750 1900 50  0001 C CNN
@@
 $EndComp
 $Comp
-L GND #PWR022
+L GND #PWR020
 U 1 1 59650F33
 P 1750 2250
-F 0 "#PWR022" H 1750 2000 50  0001 C CNN
+F 0 "#PWR020" H 1750 2000 50  0001 C CNN
 F 1 "GND" H 1750 2100 50  0000 C CNN
 F 2 "" H 1750 2250 50  0001 C CNN
@@
 Connection ~ 2100 3825
 $Comp
-L +3V3_FPGA #PWR023
+L +3V3_FPGA #PWR021
 U 1 1 5971CBE5
 P 7375 1425
-F 0 "#PWR023" H 7375 1275 50  0001 C CNN
+F 0 "#PWR021" H 7375 1275 50  0001 C CNN
 F 1 "+3V3_FPGA" H 7375 1565 50  0000 C CNN
 F 2 "" H 7375 1425 50  0001 C CNN
@@
 $EndComp
 $Comp
-L +3V6 #PWR024
+L +3V6 #PWR022
 U 1 1 597219FA
 P 5875 1125
-F 0 "#PWR024" H 5875 975 50  0001 C CNN
+F 0 "#PWR022" H 5875 975 50  0001 C CNN
 F 1 "+3V6" H 5875 1265 50  0000 C CNN
 F 2 "" H 5875 1125 50  0001 C CNN
@@
 Connection ~ 5875 1150
 Wire Wire Line
-	1275 1950 1275 1975
-Wire Wire Line
 	8400 5175 8400 5200
 Wire Wire Line
 	8600 5175 8600 5275
 $Comp
-L +3V6 #PWR025
+L +3V6 #PWR023
 U 1 1 5977DEC2
 P 8175 5150
-F 0 "#PWR025" H 8175 5000 50  0001 C CNN
+F 0 "#PWR023" H 8175 5000 50  0001 C CNN
 F 1 "+3V6" H 8175 5290 50  0000 C CNN
 F 2 "" H 8175 5150 50  0001 C CNN
@@
 	1750 1900 1750 1950
 Connection ~ 1750 1925
-Connection ~ 1275 3275
-Wire Wire Line
-	1275 3725 1275 3700
 Wire Wire Line
 	2050 1925 2050 3525
@@
 	9100 5825 9100 5800
 $Comp
-L GND #PWR026
+L GND #PWR024
 U 1 1 59E1CD41
 P 3150 5025
-F 0 "#PWR026" H 3150 4775 50  0001 C CNN
+F 0 "#PWR024" H 3150 4775 50  0001 C CNN
 F 1 "GND" H 3150 4875 50  0000 C CNN
 F 2 "" H 3150 5025 50  0001 C CNN
@@
 	1    0    0    -1
 $EndComp
+Wire Wire Line
+	1275 2575 1275 3275
 $EndSCHEMATC

Commit message: clean up in layout & add exports (assembly drawings)
Parts:
- C1, C10, C2, C3, C4, C5, C6, C7, C9: footprint Capacitors_SMD:C_0603_HandSoldering -> Footprints_LJ:Cap_0603_HandSoldering_1
Changed lines of the file:
@@
 F 0 "C1" H 8200 2125 50  0000 L CNN
 F 1 "10u" H 8200 1925 50  0000 L CNN
-F 2 "Capacitors_SMD:C_0603_HandSoldering" H 8213 1875 50  0001 C CNN
+F 2 "Footprints_LJ:Cap_0603_HandSoldering_1" H 8213 1875 50  0001 C CNN
 F 3 "" H 8175 2025 50  0001 C CNN
 	1    8175 2025
@@
 F 0 "C2" H 8550 2125 50  0000 L CNN
 F 1 "10u" H 8550 1925 50  0000 L CNN
-F 2 "Capacitors_SMD:C_0603_HandSoldering" H 8563 1875 50  0001 C CNN
+F 2 "Footprints_LJ:Cap_0603_HandSoldering_1" H 8563 1875 50  0001 C CNN
 F 3 "" H 8525 2025 50  0001 C CNN
 	1    8525 2025
@@
 F 0 "C4" H 5600 1425 50  0000 L CNN
 F 1 "10u" H 5600 1225 50  0000 L CNN
-F 2 "Capacitors_SMD:C_0603_HandSoldering" H 5613 1175 50  0001 C CNN
+F 2 "Footprints_LJ:Cap_0603_HandSoldering_1" H 5613 1175 50  0001 C CNN
 F 3 "" H 5575 1325 50  0001 C CNN
 	1    5575 1325
@@
 F 0 "C10" H 10100 5475 50  0000 L CNN
 F 1 "10u" H 10100 5275 50  0000 L CNN
-F 2 "Capacitors_SMD:C_0603_HandSoldering" H 10113 5225 50  0001 C CNN
+F 2 "Footprints_LJ:Cap_0603_HandSoldering_1" H 10113 5225 50  0001 C CNN
 F 3 "" H 10075 5375 50  0001 C CNN
 	1    10075 5375
@@
 F 0 "C5" H 6750 1725 50  0000 L CNN
 F 1 "10u" H 6750 1525 50  0000 L CNN
-F 2 "Capacitors_SMD:C_0603_HandSoldering" H 6763 1475 50  0001 C CNN
+F 2 "Footprints_LJ:Cap_0603_HandSoldering_1" H 6763 1475 50  0001 C CNN
 F 3 "" H 6725 1625 50  0001 C CNN
 	1    6725 1625
@@
 F 0 "C6" H 7100 1725 50  0000 L CNN
 F 1 "10u" H 7100 1525 50  0000 L CNN
-F 2 "Capacitors_SMD:C_0603_HandSoldering" H 7113 1475 50  0001 C CNN
+F 2 "Footprints_LJ:Cap_0603_HandSoldering_1" H 7113 1475 50  0001 C CNN
 F 3 "" H 7075 1625 50  0001 C CNN
 	1    7075 1625
@@
 F 0 "C7" H 1775 2200 50  0000 L CNN
 F 1 "100n" H 1775 2000 50  0000 L CNN
-F 2 "Capacitors_SMD:C_0603_HandSoldering" H 1788 1950 50  0001 C CNN
+F 2 "Footprints_LJ:Cap_0603_HandSoldering_1" H 1788 1950 50  0001 C CNN
 F 3 "" H 1750 2100 50  0001 C CNN
 	1    1750 2100
@@
 F 0 "C9" H 8200 5450 50  0000 L CNN
 F 1 "10u" H 8200 5250 50  0000 L CNN
-F 2 "Capacitors_SMD:C_0603_HandSoldering" H 8213 5200 50  0001 C CNN
+F 2 "Footprints_LJ:Cap_0603_HandSoldering_1" H 8213 5200 50  0001 C CNN
 F 3 "" H 8175 5350 50  0001 C CNN
 	1    8175 5350
@@
 F 0 "C3" H 5250 1425 50  0000 L CNN
 F 1 "10u" H 5250 1225 50  0000 L CNN
-F 2 "Capacitors_SMD:C_0603_HandSoldering" H 5263 1175 50  0001 C CNN
+F 2 "Footprints_LJ:Cap_0603_HandSoldering_1" H 5263 1175 50  0001 C CNN
 F 3 "" H 5225 1325 50  0001 C CNN
 	1    5225 1325
